File: Resistor_Cali/Resistor_Cali.kicad_pcb (KiCad board)
At the start: 2 copper layers, 59 parts, among them J1 DB9_Female, J2 Conn_01x20_Female, J3 Conn_01x20_Female, J4 Conn_01x01_Female, J5 Conn_Coaxial, U1 KAQY212S, U10 KAQY212S, U11 KAQY212S, U12 KAQY212S, U13 KAQY212S, U14 KAQY212S, U15 KAQY212S, U16 KAQY212S, U17 KAQY212S, U18 KAQY212S, U2 KAQY212S, U3 KAQY212S, U4 KAQY212S, U5 KAQY212S, U6 KAQY212S, U7 KAQY212S, U8 KAQY212S, U9 KAQY212S

Commit message: Update
Parts:
- added J6: Conn_01x01_Female, Connector_PinSocket_2.54mm:PinSocket_1x01_P2.54mm_Horizontal, F.Cu at (-65.1, 27.6)
- J1: value DB9_Female -> Conn_Coaxial; footprint Connector:DB9_ASSMANN -> Connector:SMA-TH_BWSMA-KE-Z001
- J2: value Conn_01x20_Female -> DB9_Female; footprint Connector_PinSocket_2.54mm:PinSocket_1x20_P2.54mm_Vertical -> Connector:DB9_ASSMANN
- J4: value Conn_01x01_Female -> Conn_01x20_Female; footprint Connector_PinSocket_2.54mm:PinSocket_1x01_P2.54mm_Horizontal -> Connector_PinSocket_2.54mm:PinSocket_1x20_P2.54mm_Vertical
- J5: value Conn_Coaxial -> Conn_01x16_Female; footprint Connector:SMA-TH_BWSMA-KE-Z001 -> Connector_PinHeader_2.54mm:PinHeader_1x16_P2.54mm_Vertical
- R1, R19: value 100K_0.1% -> 1K_1%
- R10: value 1K_1% -> 120K_0.1%
- R12, R30: value 1K_1% -> 140K_0.1%
- R13, R31: value 140K_0.1% -> 150K_0.1%; footprint Resistor_SMD:R0603 -> Resistor_SMD:150K_0.1
- R14, R32: value 1K_1% -> 160K_0.1%; footprint Resistor_SMD:R0603 -> Resistor_SMD:160K_0.1
- R15, R33: value 150K_0.1% -> 1K_1%; footprint Resistor_SMD:150K_0.1 -> Resistor_SMD:R0603
- R17, R35: value 160K_0.1% -> 180K_0.1%; footprint Resistor_SMD:160K_0.1 -> Resistor_SMD:180K_0.1
- R18, R36: value 1K_1% -> 200K_0.1%
- R2, R23: value 180K_0.1% -> 1K_1%; footprint Resistor_SMD:180K_0.1 -> Resistor_SMD:R0603
- R21, R5: value 110K_0.1% -> 1K_1%
- R25: value 120K_0.1% -> 1K_1%
- R26, R8: value 1K_1% -> 100K_0.1%
- R27: value 200K_0.1% -> 110K_0.1%
- R28: value 130K_0.1% -> 120K_0.1%
- R29: value 1K_1% -> 130K_0.1%
- R7: value 200K_0.1% -> 1K_1%
- R9: value 120K_0.1% -> 110K_0.1%
- moved J2 174.9 mm to (-63.6, 14.2), turned to 270 degrees
- moved J5 160.9 mm to (-38.1, 24.1), turned to 90 degrees
- moved J4 152.9 mm to (-0.03, 19.3), turned to 270 degrees
- moved R35 125.7 mm to (-53.5, 30.5), turned to 270 degrees
- moved J3 123.5 mm to (-0.03, 1.55), turned to 270 degrees
- moved R36 123.3 mm to (-46.5, 33.5), turned to 180 degrees
- moved R33 122.7 mm to (-48.3, 22.3), turned to 270 degrees
- moved U18 122.5 mm to (-44.5, 28.3), turned to 180 degrees
- moved U17 121.0 mm to (-49.5, 28.3), turned to 180 degrees
- moved U14 113.8 mm to (-42.0, -8.57)
- moved R34 109.6 mm to (-45.7, 22.3), turned to 270 degrees
- moved R29 109.2 mm to (-36.4, -13.6), turned to 180 degrees
- moved R23 105.8 mm to (-40.7, -1.77), turned to 90 degrees
- moved R24 105.3 mm to (-45.7, -1.77)
- moved U13 103.4 mm to (-37.0, -8.57)
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Connections:
- J1 pad 1: /I+ -> Net-(J1-Pad1)
- J1 pad 2: /I- -> GND
- J2 pad 0: /0 -> GND
- J2 pad 2: /1 -> /I-
- J2 pad 4: /2 -> /I+_2
- J2 pad 5: /3 -> /I-_2
- J2 pad 6: /4 -> /I+
- J2 pad 7: /5 -> /I-
- J2 pad 8: GND -> /I+_2
- J2 pad 9: /6 -> /I-_2
- J3 pad 1: /VBUS -> /0
- J3 pad 10: /26 -> /7
- J3 pad 11: /RUN -> /8
- J3 pad 12: /22 -> /9
- J3 pad 14: /21 -> /10
- J3 pad 15: /20 -> /11
- J3 pad 16: /19 -> /12
- J3 pad 17: /18 -> /13
- J3 pad 19: /17 -> /14
- J3 pad 2: /VSYS -> /1
- J3 pad 20: /16 -> /15
- J3 pad 4: /3V3_EN -> /2
- J3 pad 5: /3V3_OUT -> /3
- J3 pad 6: /ADC_VREF -> /4
- J3 pad 7: /28 -> /5
- J3 pad 9: /27 -> /6
- J4 pad 1: /18 -> /VBUS
- J5 pad 1: /Top Resistors/V+ -> /19
- J5 pad 2: GND -> /20
- J5 pad 3: (no net) -> /21
- J5 pad 4: (no net) -> GND
- J5 pad 5: (no net) -> /22
- R1 pad 1: /Top Resistors/V+ -> /0
- R1 pad 2: /Top Resistors/I- -> Net-(R1-Pad2)
- R10 pad 1: /Top Resistors/2 -> Net-(R10-Pad1)
- R10 pad 2: Net-(R10-Pad2) -> /I-
- R11 pad 1: /Top Resistors/V+ -> Net-(R11-Pad1)
- R11 pad 2: /Top Resistors/I- -> /I-
- R12 pad 1: /Top Resistors/3 -> Net-(R12-Pad1)
- R12 pad 2: Net-(R12-Pad2) -> /I-
- R13 pad 1: /Top Resistors/V+ -> Net-(R13-Pad1)
- R13 pad 2: /Top Resistors/I- -> /I-
- R14 pad 1: /Top Resistors/4 -> Net-(R14-Pad1)
- R14 pad 2: Net-(R14-Pad2) -> /I-
- R15 pad 1: /Top Resistors/V+ -> /7
- R15 pad 2: /Top Resistors/I- -> Net-(R15-Pad2)
- R16 pad 1: /Top Resistors/5 -> /8
- R17 pad 1: /Top Resistors/V+ -> Net-(R17-Pad1)
- R17 pad 2: /Top Resistors/I- -> /I-
- R18 pad 1: /Top Resistors/6 -> Net-(R18-Pad1)
- R18 pad 2: Net-(R18-Pad2) -> /I-
- R19 pad 1: /Bottom_Resistors/V+_2 -> /9
- R19 pad 2: /Bottom_Resistors/I-_2 -> Net-(R19-Pad2)
- R2 pad 1: /Top Resistors/V+ -> /1
- R2 pad 2: /Top Resistors/I- -> Net-(R2-Pad2)
- R20 pad 1: /Bottom_Resistors/9 -> /10
- R21 pad 1: /Bottom_Resistors/V+_2 -> /11
- R21 pad 2: /Bottom_Resistors/I-_2 -> Net-(R21-Pad2)
- R22 pad 1: /Bottom_Resistors/10 -> /12
- R23 pad 1: /Bottom_Resistors/V+_2 -> /13
- R23 pad 2: /Bottom_Resistors/I-_2 -> Net-(R23-Pad2)
- R24 pad 1: /Bottom_Resistors/16 -> /14
- R25 pad 1: /Bottom_Resistors/V+_2 -> /15
- R25 pad 2: /Bottom_Resistors/I-_2 -> Net-(R25-Pad2)
- R26 pad 1: /Bottom_Resistors/11 -> Net-(R26-Pad1)
- R26 pad 2: Net-(R26-Pad2) -> /I-_2
- R27 pad 1: /Bottom_Resistors/V+_2 -> Net-(R27-Pad1)
- R27 pad 2: /Bottom_Resistors/I-_2 -> /I-_2
- R28 pad 1: /Bottom_Resistors/V+_2 -> Net-(R28-Pad1)
- R28 pad 2: /Bottom_Resistors/I-_2 -> /I-_2
- R29 pad 1: /Bottom_Resistors/17 -> Net-(R29-Pad1)
- R29 pad 2: Net-(R29-Pad2) -> /I-_2
- R3 pad 1: /Top Resistors/0 -> /2
- R30 pad 1: /Bottom_Resistors/12 -> Net-(R30-Pad1)
- R30 pad 2: Net-(R30-Pad2) -> /I-_2
- R31 pad 1: /Bottom_Resistors/V+_2 -> Net-(R31-Pad1)
- R31 pad 2: /Bottom_Resistors/I-_2 -> /I-_2
- R32 pad 1: /Bottom_Resistors/13 -> Net-(R32-Pad1)
- R32 pad 2: Net-(R32-Pad2) -> /I-_2
- R33 pad 1: /Bottom_Resistors/V+_2 -> /16
- R33 pad 2: /Bottom_Resistors/I-_2 -> Net-(R33-Pad2)
- R34 pad 1: /Bottom_Resistors/14 -> /17
- R35 pad 1: /Bottom_Resistors/V+_2 -> Net-(R35-Pad1)
- R35 pad 2: /Bottom_Resistors/I-_2 -> /I-_2
- R36 pad 1: /Bottom_Resistors/15 -> Net-(R36-Pad1)
- R36 pad 2: Net-(R36-Pad2) -> /I-_2
- R4 pad 1: /Top Resistors/7 -> /3
- R5 pad 1: /Top Resistors/V+ -> /4
- R5 pad 2: /Top Resistors/I- -> Net-(R5-Pad2)
- R6 pad 1: /Top Resistors/1 -> /5
- R7 pad 1: /Top Resistors/V+ -> /6
- R7 pad 2: /Top Resistors/I- -> Net-(R7-Pad2)
- R8 pad 1: /Top Resistors/8 -> Net-(J1-Pad1)
- R8 pad 2: Net-(R8-Pad2) -> /I-
- R9 pad 1: /Top Resistors/V+ -> Net-(R9-Pad1)
- R9 pad 2: /Top Resistors/I- -> /I-
- U1 pad 1: Net-(R3-Pad2) -> Net-(R1-Pad2)
- U1 pad 3: /Top Resistors/V+ -> Net-(J1-Pad1)
- U1 pad 4: /Top Resistors/I+ -> /I+
- U10 pad 1: Net-(R20-Pad2) -> Net-(R19-Pad2)
- U10 pad 3: /Bottom_Resistors/V+_2 -> Net-(R26-Pad1)
- U10 pad 4: /Bottom_Resistors/I+_2 -> /I+_2
- U11 pad 1: Net-(R22-Pad2) -> Net-(R20-Pad2)
- U11 pad 3: /Bottom_Resistors/V+_2 -> Net-(R27-Pad1)
- U11 pad 4: /Bottom_Resistors/I+_2 -> /I+_2
- U12 pad 1: Net-(R24-Pad2) -> Net-(R21-Pad2)
- U12 pad 3: /Bottom_Resistors/V+_2 -> Net-(R28-Pad1)
- U12 pad 4: /Bottom_Resistors/I+_2 -> /I+_2
- U13 pad 1: Net-(R26-Pad2) -> Net-(R22-Pad2)
- U13 pad 3: /Bottom_Resistors/V+_2 -> Net-(R29-Pad1)
- U13 pad 4: /Bottom_Resistors/I+_2 -> /I+_2
- U14 pad 1: Net-(R29-Pad2) -> Net-(R23-Pad2)
- U14 pad 3: /Bottom_Resistors/V+_2 -> Net-(R30-Pad1)
- U14 pad 4: /Bottom_Resistors/I+_2 -> /I+_2
- U15 pad 1: Net-(R30-Pad2) -> Net-(R24-Pad2)
- U15 pad 3: /Bottom_Resistors/V+_2 -> Net-(R31-Pad1)
- U15 pad 4: /Bottom_Resistors/I+_2 -> /I+_2
- U16 pad 1: Net-(R32-Pad2) -> Net-(R25-Pad2)
- U16 pad 3: /Bottom_Resistors/V+_2 -> Net-(R32-Pad1)
- U16 pad 4: /Bottom_Resistors/I+_2 -> /I+_2
- U17 pad 1: Net-(R34-Pad2) -> Net-(R33-Pad2)
- U17 pad 3: /Bottom_Resistors/V+_2 -> Net-(R35-Pad1)
- U17 pad 4: /Bottom_Resistors/I+_2 -> /I+_2
- U18 pad 1: Net-(R36-Pad2) -> Net-(R34-Pad2)
- U18 pad 3: /Bottom_Resistors/V+_2 -> Net-(R36-Pad1)
- U18 pad 4: /Bottom_Resistors/I+_2 -> /I+_2
- U2 pad 1: Net-(R4-Pad2) -> Net-(R2-Pad2)
- U2 pad 3: /Top Resistors/V+ -> Net-(R9-Pad1)
- U2 pad 4: /Top Resistors/I+ -> /I+
- U3 pad 1: Net-(R6-Pad2) -> Net-(R3-Pad2)
- U3 pad 3: /Top Resistors/V+ -> Net-(R10-Pad1)
- U3 pad 4: /Top Resistors/I+ -> /I+
- U4 pad 1: Net-(R8-Pad2) -> Net-(R4-Pad2)
- U4 pad 3: /Top Resistors/V+ -> Net-(R11-Pad1)
- U4 pad 4: /Top Resistors/I+ -> /I+
- U5 pad 1: Net-(R10-Pad2) -> Net-(R5-Pad2)
- U5 pad 3: /Top Resistors/V+ -> Net-(R12-Pad1)
- U5 pad 4: /Top Resistors/I+ -> /I+
- U6 pad 1: Net-(R12-Pad2) -> Net-(R6-Pad2)
- U6 pad 3: /Top Resistors/V+ -> Net-(R13-Pad1)
- U6 pad 4: /Top Resistors/I+ -> /I+
- U7 pad 1: Net-(R14-Pad2) -> Net-(R7-Pad2)
- U7 pad 3: /Top Resistors/V+ -> Net-(R14-Pad1)
- U7 pad 4: /Top Resistors/I+ -> /I+
- U8 pad 1: Net-(R16-Pad2) -> Net-(R15-Pad2)
- U8 pad 3: /Top Resistors/V+ -> Net-(R17-Pad1)
- U8 pad 4: /Top Resistors/I+ -> /I+
- U9 pad 1: Net-(R18-Pad2) -> Net-(R16-Pad2)
- U9 pad 3: /Top Resistors/V+ -> Net-(R18-Pad1)
- U9 pad 4: /Top Resistors/I+ -> /I+
Routing:
- net /I-: track 0.00 -> 122.4 mm
- net /I+: track 0.00 -> 121.1 mm, vias 0 -> 9
- net /I-_2: track 0.00 -> 104.7 mm
- net /I+_2: track 0.00 -> 101.5 mm, vias 0 -> 9
- net /18: track 0.00 -> 39.1 mm
- net GND: track 0.00 -> 37.8 mm
- net Net-(J1-Pad1): track 0.00 -> 27.8 mm
- net Net-(R31-Pad1): track 0.00 -> 14.4 mm
- net Net-(R15-Pad2): track 0.00 -> 11.5 mm
- net Net-(R7-Pad2): track 0.00 -> 10.1 mm
- net Net-(R6-Pad2): track 0.00 -> 9.20 mm
- net Net-(R16-Pad2): track 0.00 -> 8.31 mm
- net Net-(R5-Pad2): track 0.00 -> 7.92 mm
- net Net-(R32-Pad1): track 0.00 -> 7.25 mm
- net Net-(R25-Pad2): track 0.00 -> 6.14 mm
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- added copper zone on B.Cu, net GND
- added copper zone on F.Cu, net GND
Other:
- board outline added: 77 x 50 mm
- net class Default: clearance 0.2 -> 0.25
- rule trace_clearance: 0.2 -> 0.25
- board text added: "Resistor01 Ryan Morgenstern 5/2/2021"
