File: Resistor_Cali/Resistor_Cali.sch (KiCad schematic (older format))
At the start: 30 parts

Commit message: update
Parts:
- added C?: 470nF, kicad_lceda:C0603, symbol 0_My_Lib:CL10B474KA8NNNC
- added R?: 250K_0.1%, kicad_lceda:R1206, symbol 0_My_Lib:250K_0.1%
- added U?: REF3025AIDBZR, kicad_lceda:SOT-23-3_L2.9-W1.6-P1.90-LS2.8-BR, symbol 0_My_Lib:REF3025AIDBZR
- R?: symbol 0My_Library:100K_0.1% -> Resistor_Cali-rescue:100K_0.1%-0My_Library
- R?: symbol 0My_Library:110K_0.1% -> Resistor_Cali-rescue:110K_0.1%-0My_Library
- R?: symbol 0My_Library:120K_0.1% -> Resistor_Cali-rescue:120K_0.1%-0My_Library
- R? (x9): symbol 0My_Library:1K_1% -> Resistor_Cali-rescue:1K_1%-0My_Library
- R?: symbol 0My_Library:130K_0.1% -> Resistor_Cali-rescue:130K_0.1%-0My_Library
- R?: symbol 0My_Library:140K_0.1% -> Resistor_Cali-rescue:140K_0.1%-0My_Library
- R?: symbol 0My_Library:150K_0.1% -> Resistor_Cali-rescue:150K_0.1%-0My_Library
- R?: symbol 0My_Library:160K_0.1% -> Resistor_Cali-rescue:160K_0.1%-0My_Library
- R?: symbol 0My_Library:180K_0.1% -> Resistor_Cali-rescue:180K_0.1%-0My_Library
- R?: symbol 0My_Library:200K_0.1% -> Resistor_Cali-rescue:200K_0.1%-0My_Library
- U? (x9): symbol 0My_Library:KAQY212S -> Resistor_Cali-rescue:KAQY212S-0My_Library
Connections:
- net labels added: 2.5V, VCC
- wire segments 8 -> 12
Other:
- note added: "2.5V Source to 10 uA\n"
- moved on the sheet: J?
Changed lines of the file:
@@
 $EndComp
 $Comp
-L 0My_Library:100K_0.1% R?
+L Resistor_Cali-rescue:100K_0.1%-0My_Library R?
 U 1 1 62602404
 P 2100 2250
@@
 $EndComp
 $Comp
-L 0My_Library:110K_0.1% R?
+L Resistor_Cali-rescue:110K_0.1%-0My_Library R?
 U 1 1 626031BA
 P 3200 2200
@@
 $EndComp
 $Comp
-L 0My_Library:KAQY212S U?
+L Resistor_Cali-rescue:KAQY212S-0My_Library U?
 U 1 1 6260622D
 P 2300 1500
@@
 $EndComp
 $Comp
-L 0My_Library:KAQY212S U?
+L Resistor_Cali-rescue:KAQY212S-0My_Library U?
 U 1 1 6260B48E
 P 3400 1500
@@
 L Connector:DB9_Female J?
 U 1 1 6260D163
-P 1200 2900
-F 0 "J?" H 1118 2208 50  0000 C CNN
-F 1 "DB9_Female" H 1118 2299 50  0000 C CNN
-F 2 "" H 1200 2900 50  0001 C CNN
-F 3 " ~" H 1200 2900 50  0001 C CNN
-F 4 "C75749" H 1200 2900 50  0001 C CNN "LCSC"
-	1    1200 2900
+P 800 3150
+F 0 "J?" H 718 2458 50  0000 C CNN
+F 1 "DB9_Female" H 718 2549 50  0000 C CNN
+F 2 "" H 800 3150 50  0001 C CNN
+F 3 " ~" H 800 3150 50  0001 C CNN
+F 4 "C75749" H 800 3150 50  0001 C CNN "LCSC"
+	1    800  3150
 	-1   0    0    -1
 $EndComp
 Wire Wire Line
-	1500 2500 1750 2500
-Wire Wire Line
-	1500 2600 1750 2600
-Wire Wire Line
-	1500 2700 1750 2700
-Wire Wire Line
-	1500 2800 1750 2800
+	1100 2750 1350 2750
+Wire Wire Line
+	1100 2850 1350 2850
+Wire Wire Line
+	1100 2950 1350 2950
+Wire Wire Line
+	1100 3050 1350 3050
 $Comp
 L power:GND #PWR?
 U 1 1 62615F19
-P 1500 2900
-F 0 "#PWR?" H 1500 2650 50  0001 C CNN
-F 1 "GND" V 1505 2772 50  0000 R CNN
-F 2 "" H 1500 2900 50  0001 C CNN
-F 3 "" H 1500 2900 50  0001 C CNN
-	1    1500 2900
+P 1100 3150
+F 0 "#PWR?" H 1100 2900 50  0001 C CNN
+F 1 "GND" V 1105 3022 50  0000 R CNN
+F 2 "" H 1100 3150 50  0001 C CNN
+F 3 "" H 1100 3150 50  0001 C CNN
+	1    1100 3150
 	0    -1   -1   0
 $EndComp
@@
 	0    1    1    0
 $EndComp
-Text Label 1750 2500 0    50   ~ 0
-I+
-Text Label 1100 2550 0    50   ~ 0
+Text Label 1350 2850 0    50   ~ 0
 V+
-Text Label 1750 2700 0    50   ~ 0
-I-
-Text Label 1750 2800 0    50   ~ 0
+Text Label 1350 3050 0    50   ~ 0
 V-
-NoConn ~ 1500 3000
-NoConn ~ 1500 3100
-NoConn ~ 1500 3200
+NoConn ~ 1100 3250
+NoConn ~ 1100 3350
+NoConn ~ 1100 3450
 NoConn ~ 1500 3300
 Wire Wire Line
@@
 Wire Wire Line
 	2100 2450 2100 2550
-Connection ~ 2100 2450
 Wire Wire Line
 	1850 2050 2100 2050
@@
 I-
 $Comp
-L 0My_Library:KAQY212S U?
+L Resistor_Cali-rescue:KAQY212S-0My_Library U?
 U 1 1 6261FEFE
 P 4700 1500
@@
 $EndComp
 $Comp
-L 0My_Library:KAQY212S U?
+L Resistor_Cali-rescue:KAQY212S-0My_Library U?
 U 1 1 62625B8A
 P 5850 1500
@@
 $EndComp
 $Comp
-L 0My_Library:KAQY212S U?
+L Resistor_Cali-rescue:KAQY212S-0My_Library U?
 U 1 1 62626F34
 P 6900 1500
@@
 $EndComp
 $Comp
-L 0My_Library:KAQY212S U?
+L Resistor_Cali-rescue:KAQY212S-0My_Library U?
 U 1 1 626281B2
 P 8000 1500
@@
 $EndComp
 $Comp
-L 0My_Library:KAQY212S U?
+L Resistor_Cali-rescue:KAQY212S-0My_Library U?
 U 1 1 62629EB9
 P 9150 1500
@@
 $EndComp
 $Comp
-L 0My_Library:KAQY212S U?
+L Resistor_Cali-rescue:KAQY212S-0My_Library U?
 U 1 1 6262AB1E
 P 10250 1500
@@
 $EndComp
 $Comp
-L 0My_Library:120K_0.1% R?
+L Resistor_Cali-rescue:120K_0.1%-0My_Library R?
 U 1 1 6263C8D6
 P 4500 2200
@@
 $EndComp
 $Comp
-L 0My_Library:1K_1% R?
+L Resistor_Cali-rescue:1K_1%-0My_Library R?
 U 1 1 6263F9C0
 P 2500 800
@@
 $EndComp
 $Comp
-L 0My_Library:1K_1% R?
+L Resistor_Cali-rescue:1K_1%-0My_Library R?
 U 1 1 62640D00
 P 3600 800
@@
 $EndComp
 $Comp
-L 0My_Library:1K_1% R?
+L Resistor_Cali-rescue:1K_1%-0My_Library R?
 U 1 1 6264118F
 P 4900 800
@@
 $EndComp
 $Comp
-L 0My_Library:1K_1% R?
+L Resistor_Cali-rescue:1K_1%-0My_Library R?
 U 1 1 626415F5
 P 6050 800
@@
 $EndComp
 $Comp
-L 0My_Library:1K_1% R?
+L Resistor_Cali-rescue:1K_1%-0My_Library R?
 U 1 1 62641A26
 P 7100 800
@@
 $EndComp
 $Comp
-L 0My_Library:1K_1% R?
+L Resistor_Cali-rescue:1K_1%-0My_Library R?
 U 1 1 626427B4
 P 8200 800
@@
 $EndComp
 $Comp
-L 0My_Library:130K_0.1% R?
+L Resistor_Cali-rescue:130K_0.1%-0My_Library R?
 U 1 1 62642D75
 P 5650 2200
@@
 $EndComp
 $Comp
-L 0My_Library:140K_0.1% R?
+L Resistor_Cali-rescue:140K_0.1%-0My_Library R?
 U 1 1 626439B0
 P 6700 2200
@@
 $EndComp
 $Comp
-L 0My_Library:150K_0.1% R?
+L Resistor_Cali-rescue:150K_0.1%-0My_Library R?
 U 1 1 62644760
 P 7800 2200
@@
 $EndComp
 $Comp
-L 0My_Library:160K_0.1% R?
+L Resistor_Cali-rescue:160K_0.1%-0My_Library R?
 U 1 1 626456B0
 P 8950 2200
@@
 $EndComp
 $Comp
-L 0My_Library:180K_0.1% R?
+L Resistor_Cali-rescue:180K_0.1%-0My_Library R?
 U 1 1 62646B04
 P 10050 2200
@@
 $EndComp
 $Comp
-L 0My_Library:200K_0.1% R?
+L Resistor_Cali-rescue:200K_0.1%-0My_Library R?
 U 1 1 626478D6
 P 10050 4250
@@
 $EndComp
 $Comp
-L 0My_Library:KAQY212S U?
+L Resistor_Cali-rescue:KAQY212S-0My_Library U?
 U 1 1 6264B9E6
 P 10250 3550
@@
 $EndComp
 $Comp
-L 0My_Library:1K_1% R?
+L Resistor_Cali-rescue:1K_1%-0My_Library R?
 U 1 1 6264B9EE
 P 10450 2850
@@
 $EndComp
 $Comp
-L 0My_Library:1K_1% R?
+L Resistor_Cali-rescue:1K_1%-0My_Library R?
 U 1 1 6264C25C
 P 10450 800
@@
 $EndComp
 $Comp
-L 0My_Library:1K_1% R?
+L Resistor_Cali-rescue:1K_1%-0My_Library R?
 U 1 1 6264C720
 P 9350 800
@@
 	0    1    1    0
 $EndComp
+Wire Notes Line
+	600  5950 600  7750
+Wire Notes Line
+	600  7750 3450 7750
+Wire Notes Line
+	3450 5950 600  5950
+Wire Notes Line
+	3450 5950 3450 7750
+Text Notes 1500 6050 0    50   ~ 0
+2.5V Source to 10 uA\n
+$Comp
+L 0_My_Lib:CL10B474KA8NNNC C?
+U 1 1 62675DD8
+P 1600 7600
+F 0 "C?" H 1600 7355 50  0000 C CNN
+F 1 "470nF" H 1600 7446 50  0000 C CNN
+F 2 "kicad_lceda:C0603" H 1600 7580 50  0001 C CNN
+F 3 "http://www.szlcsc.com/product/details_1975.html" H 1600 7380 50  0001 C CNN
+F 4 "C1623" H 1600 7180 50  0001 C CNN "LCSC"
+F 5 "std:b9126dca6316fd5ce40a4f870ab302ac" H 1600 7180 50  0001 C CNN "uuid"
+	1    1600 7600
+	1    0    0    1
+$EndComp
+$Comp
+L 0_My_Lib:REF3025AIDBZR U?
+U 1 1 62678AA9
+P 2050 7100
+F 0 "U?" H 2050 7465 50  0000 C CNN
+F 1 "REF3025AIDBZR" H 2050 7374 50  0000 C CNN
+F 2 "kicad_lceda:SOT-23-3_L2.9-W1.6-P1.90-LS2.8-BR" H 2050 7200 50  0001 C CNN
+F 3 "http://www.szlcsc.com/product/details_11887.html" H 2050 7000 50  0001 C CNN
+F 4 "C11334" H 2050 6800 50  0001 C CNN "LCSC"
+F 5 "std:4af85dda741faa60d87c85486a4e536b" H 2050 6800 50  0001 C CNN "uuid"
+	1    2050 7100
+	1    0    0    -1
+$EndComp
+Wire Wire Line
+	1550 7000 1450 7000
+Wire Wire Line
+	1450 7000 1450 7600
+Wire Wire Line
+	1750 7600 2550 7600
+Wire Wire Line
+	2550 7600 2550 7200
+$Comp
+L power:GND #PWR?
+U 1 1 6267E0A8
+P 2550 7200
+F 0 "#PWR?" H 2550 6950 50  0001 C CNN
+F 1 "GND" V 2555 7072 50  0000 R CNN
+F 2 "" H 2550 7200 50  0001 C CNN
+F 3 "" H 2550 7200 50  0001 C CNN
+	1    2550 7200
+	0    -1   -1   0
+$EndComp
+Connection ~ 2550 7200
+Text Label 2550 7000 0    50   ~ 0
+2.5V
+Text Label 1450 7000 0    50   ~ 0
+VCC
+$Comp
+L 0_My_Lib:250K_0.1% R?
+U 1 1 626810B4
+P 1750 6450
+F 0 "R?" H 1750 6655 50  0000 C CNN
+F 1 "250K_0.1%" H 1750 6564 50  0000 C CNN
+F 2 "kicad_lceda:R1206" H 1750 6390 50  0001 C CNN
+F 3 "http://www.szlcsc.com/product/details_346873.html" H 1750 6190 50  0001 C CNN
+F 4 "C374782" H 1750 5990 50  0001 C CNN "SuppliersPartNumber"
+F 5 "std:cb5ced8bd30f43ce8de2fd2eca084dc1" H 1750 5990 50  0001 C CNN "uuid"
+	1    1750 6450
+	1    0    0    -1
+$EndComp
+Text Label 1550 6450 2    50   ~ 0
+2.5V
+Text Label 1950 6450 0    50   ~ 0
+I+
+Connection ~ 2100 2450
 $EndSCHEMATC

Commit message: update
Parts:
- removed C?: 470nF, kicad_lceda:C0603, symbol 0_My_Lib:CL10B474KA8NNNC
- removed J? (x2): Conn_01x07_Female, symbol Connector:Conn_01x07_Female
- removed R?: 100K_0.1%, kicad_lceda:R0603, symbol Resistor_Cali-rescue:100K_0.1%-0My_Library
- removed R?: 110K_0.1%, kicad_lceda:R0603, symbol Resistor_Cali-rescue:110K_0.1%-0My_Library
- removed R?: 120K_0.1%, kicad_lceda:R0603, symbol Resistor_Cali-rescue:120K_0.1%-0My_Library
- removed R? (x9): 1K_1%, kicad_lceda:R0603, symbol Resistor_Cali-rescue:1K_1%-0My_Library
- removed R?: 130K_0.1%, kicad_lceda:R0603, symbol Resistor_Cali-rescue:130K_0.1%-0My_Library
- removed R?: 140K_0.1%, kicad_lceda:R0603, symbol Resistor_Cali-rescue:140K_0.1%-0My_Library
- removed R?: 150K_0.1%, kicad_lceda:R0805, symbol Resistor_Cali-rescue:150K_0.1%-0My_Library
- removed R?: 160K_0.1%, kicad_lceda:R0805, symbol Resistor_Cali-rescue:160K_0.1%-0My_Library
- removed R?: 180K_0.1%, kicad_lceda:R0805, symbol Resistor_Cali-rescue:180K_0.1%-0My_Library
- removed R?: 200K_0.1%, kicad_lceda:R0603, symbol Resistor_Cali-rescue:200K_0.1%-0My_Library
- removed R?: 250K_0.1%, kicad_lceda:R1206, symbol 0_My_Lib:250K_0.1%
- removed U? (x9): KAQY212S, kicad_lceda:SOP-4_L4.4-W4.0-P2.54-LS7.0-BL, symbol Resistor_Cali-rescue:KAQY212S-0My_Library
- removed U?: REF3025AIDBZR, kicad_lceda:SOT-23-3_L2.9-W1.6-P1.90-LS2.8-BR, symbol 0_My_Lib:REF3025AIDBZR
- added J2, J3: Conn_01x20_Female, Connector_PinSocket_2.54mm:PinSocket_1x20_P2.54mm_Vertical, symbol Connector:Conn_01x20_Female
- added J4: Conn_01x01_Female, Connector_PinSocket_2.54mm:PinSocket_1x01_P2.54mm_Horizontal, symbol Connector:Conn_01x01_Female
- J1: renamed from J?; footprint (none) -> Connector:DB9_ASSMANN
Connections:
- net labels added: 0, 1, 10, 11, 12, 13, 14, 15, 16, 17, 18, 19, 2, 20, 21, 22, 26, 27, 28, 3, 3V3_EN, 3V3_OUT, 4, 5, 6, 7, 8, 9, ADC_VREF, I+_2, I-_2, RUN, V+_2, V-_2, VBUS, VSYS
- net labels removed: 2.5V, VCC
- wire segments 12 -> 9
- no-connect marks 4 -> 0
Other:
- note added: "Drdy Rdy \n"
- note removed: "2.5V Source to 10 uA\n"
- moved on the sheet: J1

Commit message: Update
Parts:
- added J1: Conn_Coaxial, Connector:SMA-TH_BWSMA-KE-Z001, symbol Connector:Conn_Coaxial
- added J5: Conn_01x16_Female, Connector_PinHeader_2.54mm:PinHeader_1x16_P2.54mm_Vertical, symbol Connector:Conn_01x16_Female
- added R1, R15, R16, R19, R2, R20, R21, R22, R23, R24, R25, R3, R33, R34, R4, R5, R6, R7: 1K_1%, Resistor_SMD:R0603, symbol Resistor_Cali-rescue:1K_1%-0My_Library
- added R10, R28: 120K_0.1%, Resistor_SMD:R0603, symbol Resistor_Cali-rescue:120K_0.1%-0My_Library
- added R11, R29: 130K_0.1%, Resistor_SMD:R0603, symbol Resistor_Cali-rescue:130K_0.1%-0My_Library
- added R12, R30: 140K_0.1%, Resistor_SMD:R0603, symbol Resistor_Cali-rescue:140K_0.1%-0My_Library
- added R13, R31: 150K_0.1%, Resistor_SMD:150K_0.1, symbol Resistor_Cali-rescue:150K_0.1%-0My_Library
- added R14, R32: 160K_0.1%, Resistor_SMD:160K_0.1, symbol Resistor_Cali-rescue:160K_0.1%-0My_Library
- added R17, R35: 180K_0.1%, Resistor_SMD:180K_0.1, symbol Resistor_Cali-rescue:180K_0.1%-0My_Library
- added R18, R36: 200K_0.1%, Resistor_SMD:R0603, symbol Resistor_Cali-rescue:200K_0.1%-0My_Library
- added R26, R8: 100K_0.1%, Resistor_SMD:R0603, symbol Resistor_Cali-rescue:100K_0.1%-0My_Library
- added R27, R9: 110K_0.1%, Resistor_SMD:R0603, symbol Resistor_Cali-rescue:110K_0.1%-0My_Library
- added U1, U10, U11, U12, U13, U14, U15, U16, U17, U18, U2, U3, U4, U5, U6, U7, U8, U9: KAQY212S, Connector:SOP-4_L4.4-W4.0-P2.54-LS7.0-BL, symbol Resistor_Cali-rescue:KAQY212S-0My_Library
- renumbered J1 to J2, J2 to J3, J3 to J4, J4 to J6
Connections:
- net V+ is gone; now on net I+: J2.6
- net V+_2 is gone; now on net I+_2: J2.4
- net V- is gone; now on net I-: J2.7
- net V-_2 is gone; now on net I-_2: J2.5
- net 0: now also R1.1
- net 1: now also R2.1
- net 10: now also R20.1
- net 11: now also R21.1
- net 12: now also R22.1
- net 13: now also R23.1
- net 14: now also R24.1
- net 15: now also R25.1
- net 16: now also R33.1
- net 17: now also R34.1
- net 19: now also J5.1 (Pin_1)
- net 2: now also R3.1
- net 20: now also J5.2 (Pin_2)
- net 21: now also J5.3 (Pin_3)
- net 22: now also J5.5 (Pin_5)
- net 26: now also J5.7 (Pin_7)
- net 27: now also J5.8 (Pin_8)
- net 28: now also J5.10 (Pin_10)
- net 3: now also R4.1
- net 3V3_EN: now also J5.13 (Pin_13)
- net 3V3_OUT: now also J5.12 (Pin_12)
- net 4: now also R5.1
- net 5: now also R6.1
- net 6: now also R7.1
- net 7: now also R15.1
- net 8: now also R16.1
- net 9: now also R19.1
- net ADC_VREF: now also J5.11 (Pin_11)
- net GND: now also J1.2 (Ext), J5.14 (Pin_14), J5.4 (Pin_4), J5.9 (Pin_9), U1.2, U10.2, U11.2, U12.2, U13.2, U14.2, U15.2, U16.2, U17.2, U18.2, U2.2, U3.2, U4.2, U5.2, U6.2, U7.2, U8.2, U9.2
- net I+: now also U1.4, U2.4, U3.4, U4.4, U5.4, U6.4, U7.4, U8.4, U9.4
- net I+_2: now also U10.4, U11.4, U12.4, U13.4, U14.4, U15.4, U16.4, U17.4, U18.4
- net I-: now also R10.2, R11.2, R12.2, R13.2, R14.2, R17.2, R18.2, R8.2, R9.2
- net I-_2: now also R26.2, R27.2, R28.2, R29.2, R30.2, R31.2, R32.2, R35.2, R36.2
- net RUN: now also J5.6 (Pin_6)
- net VBUS: now also J5.16 (Pin_16)
- net VSYS: now also J5.15 (Pin_15)
- new net: J1.1 (In), R8.1, U1.3
- new net: R9.1, U2.3
- new net: R1.2, U1.1
- new net: R10.1, U3.3
- new net: R11.1, U4.3
- new net: R12.1, U5.3
- new net: R13.1, U6.3
- new net: R14.1, U7.3
- new net: R2.2, U2.1
- new net: R3.2, U3.1
- new net: R4.2, U4.1
- new net: R5.2, U5.1
- new net: R6.2, U6.1
- new net: R7.2, U7.1
- new net: R16.2, U9.1
- new net: R18.1, U9.3
- new net: R15.2, U8.1
- new net: R17.1, U8.3
- new net: R26.1, U10.3
- new net: R27.1, U11.3
- new net: R19.2, U10.1
- new net: R28.1, U12.3
- new net: R29.1, U13.3
- new net: R30.1, U14.3
- new net: R31.1, U15.3
- new net: R32.1, U16.3
- new net: R36.1, U18.3
- new net: R35.1, U17.3
- new net: R20.2, U11.1
- new net: R21.2, U12.1
- new net: R22.2, U13.1
- new net: R23.2, U14.1
- new net: R24.2, U15.1
- new net: R25.2, U16.1
- new net: R33.2, U17.1
- new net: R34.2, U18.1
Other:
- moved on the sheet: J2, J3, J4, J6
