File: Resistor_02/Resistor_02/Resistor_02.sch (KiCad schematic (older format))
At the start: 17 parts

Commit message: Update
Parts:
- D1: renamed from D?; footprint (none) -> JST_Footprint_Lib:JST_SH_BM04B-SRSS-TB_1x04-1MP_P1.00mm_Vertical
- U1: renamed from U?; footprint kicad_lceda:CONN-SMD_A1001WR-S-04PD01 -> JST_Footprint_Lib:JST_SH_BM04B-SRSS-TB_1x04-1MP_P1.00mm_Vertical
- gave numbers to parts that had none: 15
Changed lines of the file:
@@
 $EndDescr
 $Comp
-L power:GND #PWR?
+L power:GND #PWR0101
 U 1 1 62741AB5
 P 7150 4600
-F 0 "#PWR?" H 7150 4350 50  0001 C CNN
+F 0 "#PWR0101" H 7150 4350 50  0001 C CNN
 F 1 "GND" H 7155 4427 50  0000 C CNN
 F 2 "" H 7150 4600 50  0001 C CNN
@@
 $EndComp
 $Comp
-L power:+3.3V #PWR?
+L power:+3.3V #PWR0102
 U 1 1 627485C7
 P 1950 4600
-F 0 "#PWR?" H 1950 4450 50  0001 C CNN
+F 0 "#PWR0102" H 1950 4450 50  0001 C CNN
 F 1 "+3.3V" H 1965 4773 50  0000 C CNN
 F 2 "" H 1950 4600 50  0001 C CNN
@@
 	1950 4600 1750 4600
 $Comp
-L power:+3.3V #PWR?
+L power:+3.3V #PWR0103
 U 1 1 6274D25F
 P 2100 5350
-F 0 "#PWR?" H 2100 5200 50  0001 C CNN
+F 0 "#PWR0103" H 2100 5200 50  0001 C CNN
 F 1 "+3.3V" H 2115 5523 50  0000 C CNN
 F 2 "" H 2100 5350 50  0001 C CNN
@@
 $EndComp
 $Comp
-L power:+3.3V #PWR?
+L power:+3.3V #PWR0104
 U 1 1 6274DA20
 P 1800 5200
-F 0 "#PWR?" H 1800 5050 50  0001 C CNN
+F 0 "#PWR0104" H 1800 5050 50  0001 C CNN
 F 1 "+3.3V" H 1815 5373 50  0000 C CNN
 F 2 "" H 1800 5200 50  0001 C CNN
@@
 $EndComp
 $Comp
-L power:GND #PWR?
+L power:GND #PWR0105
 U 1 1 6274F303
 P 4150 4700
-F 0 "#PWR?" H 4150 4450 50  0001 C CNN
+F 0 "#PWR0105" H 4150 4450 50  0001 C CNN
 F 1 "GND" V 4155 4572 50  0000 R CNN
 F 2 "" H 4150 4700 50  0001 C CNN
@@
 $EndComp
 $Comp
-L power:GND #PWR?
+L power:GND #PWR0106
 U 1 1 6274F916
 P 4150 5300
-F 0 "#PWR?" H 4150 5050 50  0001 C CNN
+F 0 "#PWR0106" H 4150 5050 50  0001 C CNN
 F 1 "GND" V 4155 5172 50  0000 R CNN
 F 2 "" H 4150 5300 50  0001 C CNN
@@
 	4150 4700 4150 4600
 $Comp
-L Connector:DB9_Female_MountingHoles J?
+L Connector:DB9_Female_MountingHoles J2
 U 1 1 6276A70E
 P 3550 3100
-F 0 "J?" H 3468 3792 50  0000 C CNN
+F 0 "J2" H 3468 3792 50  0000 C CNN
 F 1 "DB9_Female_MountingHoles" H 3468 3701 50  0000 C CNN
 F 2 "" H 3550 3100 50  0001 C CNN
@@
 V_2-
 $Comp
-L power:GND #PWR?
+L power:GND #PWR0107
 U 1 1 62781560
 P 3850 3100
-F 0 "#PWR?" H 3850 2850 50  0001 C CNN
+F 0 "#PWR0107" H 3850 2850 50  0001 C CNN
 F 1 "GND" V 3855 2972 50  0000 R CNN
 F 2 "" H 3850 3100 50  0001 C CNN
@@
 	1750 4800 1800 4800
 $Comp
-L 0_Resistor02:PCA9554PW,118_I2C_bus U?
+L 0_Resistor02:PCA9554PW,118_I2C_bus U2
 U 1 1 627E0A72
 P 3750 4950
-F 0 "U?" H 3750 5585 50  0000 C CNN
+F 0 "U2" H 3750 5585 50  0000 C CNN
 F 1 "PCA9554PW,118_I2C_bus" H 3750 5494 50  0000 C CNN
 F 2 "kicad_lceda:TSSOP-16_L5.0-W4.4-P0.65-LS6.4-BL" H 3750 6000 50  0001 C CNN
@@
 $EndComp
 $Comp
-L 0_Resistor02:10K_1% R?
+L 0_Resistor02:10K_1% R2
 U 1 1 627E1937
 P 2100 5150
-F 0 "R?" H 2100 5355 50  0000 C CNN
+F 0 "R2" H 2100 5355 50  0000 C CNN
 F 1 "10K_1%" H 2100 5264 50  0000 C CNN
 F 2 "kicad_lceda:R1206" H 2100 5090 50  0001 C CNN
@@
 $EndComp
 $Comp
-L 0_Resistor02:A1001WR-S-04PD01 U?
+L 0_Resistor02:A1001WR-S-04PD01 U1
 U 1 1 627E33B5
 P 1550 4650
-F 0 "U?" H 1778 4721 50  0000 L CNN
+F 0 "U1" H 1778 4721 50  0000 L CNN
 F 1 "A1001WR-S-04PD01" H 1778 4630 50  0000 L CNN
-F 2 "kicad_lceda:CONN-SMD_A1001WR-S-04PD01" H 1550 4920 50  0001 C CNN
+F 2 "JST_Footprint_Lib:JST_SH_BM04B-SRSS-TB_1x04-1MP_P1.00mm_Vertical" H 1550 4920 50  0001 C CNN
 F 3 "http://www.szlcsc.com/product/details_345092.html" H 1550 4720 50  0001 C CNN
 F 4 "C371571" H 1550 4520 50  0001 C CNN "LCSC"
@@
 $EndComp
 $Comp
-L Device:LED D?
+L Device:LED D1
 U 1 1 627E47A6
 P 6550 4750
-F 0 "D?" H 6543 4967 50  0000 C CNN
+F 0 "D1" H 6543 4967 50  0000 C CNN
 F 1 "LED" H 6543 4876 50  0000 C CNN
-F 2 "" H 6550 4750 50  0001 C CNN
+F 2 "JST_Footprint_Lib:JST_SH_BM04B-SRSS-TB_1x04-1MP_P1.00mm_Vertical" H 6550 4750 50  0001 C CNN
 F 3 "~" H 6550 4750 50  0001 C CNN
 F 4 "C125093" H 6550 4750 50  0001 C CNN "LCSC"
@@
 $EndComp
 $Comp
-L power:GNDS #PWR?
+L power:GNDS #PWR0108
 U 1 1 627EB0D0
 P 1400 4300
-F 0 "#PWR?" H 1400 4050 50  0001 C CNN
+F 0 "#PWR0108" H 1400 4050 50  0001 C CNN
 F 1 "GNDS" H 1405 4127 50  0000 C CNN
 F 2 "" H 1400 4300 50  0001 C CNN
@@
 $EndComp
 $Comp
-L power:GNDS #PWR?
+L power:GNDS #PWR0109
 U 1 1 627ED008
 P 1400 4950
-F 0 "#PWR?" H 1400 4700 50  0001 C CNN
+F 0 "#PWR0109" H 1400 4700 50  0001 C CNN
 F 1 "GNDS" H 1405 4777 50  0000 C CNN
 F 2 "" H 1400 4950 50  0001 C CNN
@@
 $EndComp
 $Comp
-L power:GND #PWR?
+L power:GND #PWR0110
 U 1 1 627ED8FC
 P 1750 4500
-F 0 "#PWR?" H 1750 4250 50  0001 C CNN
+F 0 "#PWR0110" H 1750 4250 50  0001 C CNN
 F 1 "GND" H 1755 4327 50  0000 C CNN
 F 2 "" H 1750 4500 50  0001 C CNN
@@
 $EndComp
 $Comp
-L power:GNDS #PWR?
+L power:GNDS #PWR0111
 U 1 1 627EED50
 P 3550 3700
-F 0 "#PWR?" H 3550 3450 50  0001 C CNN
+F 0 "#PWR0111" H 3550 3450 50  0001 C CNN
 F 1 "GNDS" H 3555 3527 50  0000 C CNN
 F 2 "" H 3550 3700 50  0001 C CNN
@@
 $EndComp
 $Comp
-L 0_Resistor02:KAQY214STLD U?
+L 0_Resistor02:KAQY214STLD U5
 U 1 1 627EFDA7
 P 6850 2200
-F 0 "U?" V 6804 2628 50  0000 L CNN
+F 0 "U5" V 6804 2628 50  0000 L CNN
 F 1 "KAQY214STLD" V 6895 2628 50  0000 L CNN
 F 2 "kicad_lceda:SOP-4_L3.9-W4.4-P2.54-LS7.0-BR" H 6850 2505 50  0001 C CNN
@@
 $EndComp
 $Comp
-L 0_Resistor02:KAQY214STLD U?
+L 0_Resistor02:KAQY214STLD U6
 U 1 1 627F53B1
 P 6850 4050
-F 0 "U?" V 6804 4478 50  0000 L CNN
+F 0 "U6" V 6804 4478 50  0000 L CNN
 F 1 "KAQY214STLD" V 6895 4478 50  0000 L CNN
 F 2 "kicad_lceda:SOP-4_L3.9-W4.4-P2.54-LS7.0-BR" H 6850 4355 50  0001 C CNN
@@
 $EndComp
 $Comp
-L Device:R R?
+L Device:R R6
 U 1 1 627F6408
 P 6550 5050
-F 0 "R?" H 6620 5096 50  0000 L CNN
+F 0 "R6" H 6620 5096 50  0000 L CNN
 F 1 "50_1%" H 6620 5005 50  0000 L CNN
 F 2 "" V 6480 5050 50  0001 C CNN
@@
 $EndComp
 $Comp
-L Connector:Conn_01x01_Female J?
+L Connector:Conn_01x01_Female J1
 U 1 1 627F98CB
 P 2450 4900
-F 0 "J?" H 2400 5050 50  0000 C CNN
+F 0 "J1" H 2400 5050 50  0000 C CNN
 F 1 "Conn_01x01_Female" H 2350 5000 50  0000 C CNN
 F 2 "" H 2450 4900 50  0001 C CNN
@@
 $EndComp
 $Comp
-L Device:LED D?
+L Device:LED D2
 U 1 1 627FE906
 P 7150 1500
-F 0 "D?" H 7143 1717 50  0000 C CNN
+F 0 "D2" H 7143 1717 50  0000 C CNN
 F 1 "LED" H 7143 1626 50  0000 C CNN
 F 2 "" H 7150 1500 50  0001 C CNN
@@
 $EndComp
 $Comp
-L Device:R R?
+L Device:R R7
 U 1 1 627FE90D
 P 7150 1200
-F 0 "R?" H 7220 1246 50  0000 L CNN
+F 0 "R7" H 7220 1246 50  0000 L CNN
 F 1 "50_1%" H 7220 1155 50  0000 L CNN
 F 2 "" V 7080 1200 50  0001 C CNN
@@
 I_01
 $Comp
-L power:GND #PWR?
+L power:GND #PWR0112
 U 1 1 6280057F
 P 6550 1650
-F 0 "#PWR?" H 6550 1400 50  0001 C CNN
+F 0 "#PWR0112" H 6550 1400 50  0001 C CNN
 F 1 "GND" V 6555 1522 50  0000 R CNN
 F 2 "" H 6550 1650 50  0001 C CNN
@@
 I_01
 $Comp
-L 0_Resistor02:10K_1% R?
+L 0_Resistor02:10K_1% R1
 U 1 1 62835B78
 P 1800 5000
-F 0 "R?" V 1754 5068 50  0000 L CNN
+F 0 "R1" V 1754 5068 50  0000 L CNN
 F 1 "10K_1%" V 1845 5068 50  0000 L CNN
 F 2 "kicad_lceda:R1206" H 1800 4940 50  0001 C CNN
@@
 Connection ~ 1800 4800
 $Comp
-L 0_Resistor02:10K_1% R?
+L 0_Resistor02:10K_1% R3
 U 1 1 62838D5E
 P 2700 5100
-F 0 "R?" V 2654 5168 50  0000 L CNN
+F 0 "R3" V 2654 5168 50  0000 L CNN
 F 1 "10K_1%" V 2745 5168 50  0000 L CNN
 F 2 "kicad_lceda:R1206" H 2700 5040 50  0001 C CNN
@@
 	2700 4900 2650 4900
 $Comp
-L power:+3.3V #PWR?
+L power:+3.3V #PWR0113
 U 1 1 6283A97E
 P 2700 5300
-F 0 "#PWR?" H 2700 5150 50  0001 C CNN
+F 0 "#PWR0113" H 2700 5150 50  0001 C CNN
 F 1 "+3.3V" H 2715 5473 50  0000 C CNN
 F 2 "" H 2700 5300 50  0001 C CNN
@@
 $EndSheet
 $Comp
-L 0_Resistor02:KAQY214STLD U?
+L 0_Resistor02:KAQY214STLD U4
 U 1 1 6284A91F
 P 5050 4050
-F 0 "U?" V 5004 4478 50  0000 L CNN
+F 0 "U4" V 5004 4478 50  0000 L CNN
 F 1 "KAQY214STLD" V 5095 4478 50  0000 L CNN
 F 2 "kicad_lceda:SOP-4_L3.9-W4.4-P2.54-LS7.0-BR" H 5050 4355 50  0001 C CNN
@@
 Connection ~ 4750 3500
 $Comp
-L 0_Resistor02:KAQY214STLD U?
+L 0_Resistor02:KAQY214STLD U3
 U 1 1 62863A00
 P 5050 2150
-F 0 "U?" V 5004 2578 50  0000 L CNN
+F 0 "U3" V 5004 2578 50  0000 L CNN
 F 1 "KAQY214STLD" V 5095 2578 50  0000 L CNN
 F 2 "kicad_lceda:SOP-4_L3.9-W4.4-P2.54-LS7.0-BR" H 5050 2455 50  0001 C CNN
@@
 	5350 3150 5350 3500
 $Comp
-L Device:R R?
+L Device:R R4
 U 1 1 628783F5
 P 4750 4750
-F 0 "R?" H 4820 4796 50  0000 L CNN
+F 0 "R4" H 4820 4796 50  0000 L CNN
 F 1 "330" H 4820 4705 50  0000 L CNN
 F 2 "" V 4680 4750 50  0001 C CNN
@@
 I_01
 $Comp
-L Device:R R?
+L Device:R R5
 U 1 1 62879439
 P 5350 1450
-F 0 "R?" H 5420 1496 50  0000 L CNN
+F 0 "R5" H 5420 1496 50  0000 L CNN
 F 1 "50_1%" H 5420 1405 50  0000 L CNN
 F 2 "" V 5280 1450 50  0001 C CNN
@@
 I_00
 $Comp
-L power:GND #PWR?
+L power:GND #PWR0114
 U 1 1 62879B17
 P 4750 1600
-F 0 "#PWR?" H 4750 1350 50  0001 C CNN
+F 0 "#PWR0114" H 4750 1350 50  0001 C CNN
 F 1 "GND" V 4755 1472 50  0000 R CNN
 F 2 "" H 4750 1600 50  0001 C CNN
@@
 $EndComp
 $Comp
-L power:GND #PWR?
+L power:GND #PWR0115
 U 1 1 6287A5D2
 P 5350 4600
-F 0 "#PWR?" H 5350 4350 50  0001 C CNN
+F 0 "#PWR0115" H 5350 4350 50  0001 C CNN
 F 1 "GND" V 5355 4472 50  0000 R CNN
 F 2 "" H 5350 4600 50  0001 C CNN
@@
 Text Label 9000 4100 2    50   ~ 0
 I_07
+$Comp
+L power:+3.3V #PWR0122
+U 1 1 628DDA57
+P 1350 5500
+F 0 "#PWR0122" H 1350 5350 50  0001 C CNN
+F 1 "+3.3V" H 1365 5673 50  0000 C CNN
+F 2 "" H 1350 5500 50  0001 C CNN
+F 3 "" H 1350 5500 50  0001 C CNN
+	1    1350 5500
+	-1   0    0    1
+$EndComp
+$Comp
+L power:PWR_FLAG #FLG0101
+U 1 1 628DE107
+P 1350 5500
+F 0 "#FLG0101" H 1350 5575 50  0001 C CNN
+F 1 "PWR_FLAG" H 1350 5673 50  0000 C CNN
+F 2 "" H 1350 5500 50  0001 C CNN
+F 3 "~" H 1350 5500 50  0001 C CNN
+	1    1350 5500
+	1    0    0    -1
+$EndComp
 $EndSCHEMATC

Commit message: Upddate
Parts:
- removed D1: LED, JST_Footprint_Lib:JST_SH_BM04B-SRSS-TB_1x04-1MP_P1.00mm_Vertical, symbol Device:LED
- removed D2: LED, symbol Device:LED
- removed R6: 50_1%, symbol Device:R
- added R1, R2, R3, R4, R8: 330, symbol Device:R
- added U1, U2, U5, U8: KAQY214STLD, kicad_lceda:SOP-4_L3.9-W4.4-P2.54-LS7.0-BR, symbol 0_Resistor02:KAQY214STLD
- R5, R7: value 50_1% -> 330; LCSC C2759402 -> C125768
- renumbered J2 to J1, J1 to J2, R3 to R10, R2 to R11, R4 to R6, R1 to R9, U2 to U10, U5 to U4, U4 to U6, U6 to U7, U1 to U9
Connections:
- wire segments 36 -> 47
Other:
- moved on the sheet: J1, J2, R10, R11, R6, R9, U10, U3, U4, U6, U7, U9
