File: Resistor_02/Resistor_02/_autosave-Resistor_02.sch (KiCad schematic (older format))
At the start: 16 parts, among them J1 Conn_01x01_Female, J2 DB9_Female_MountingHoles, U1 A1001WR-S-04PD01, U2 PCA9554PW,118_I2C_bus, U3 KAQY214STLD, U4 KAQY214STLD, U5 KAQY214STLD, U6 KAQY214STLD

Commit message: Upddate
Parts:
- added R1, R2, R3, R4, R5, R7, R8: 330, symbol Device:R
- gave numbers to parts that had none: 4
- renumbered J2 to J1, J1 to J2, R3 to R10, R2 to R11, R4 to R6, R1 to R9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
Connections:
- wire segments 34 -> 47
