File: Resistor_02/Resistor_02/_autosave-Resistor_Network.sch (KiCad schematic (older format))
At the start: 24 parts, among them U10 KAQY214STLD, U11 KAQY214STLD, U12 KAQY214STLD, U7 KAQY214STLD, U8 KAQY214STLD, U9 KAQY214STLD

Commit message: Upddate
Parts:
- removed D? (x6): LED, JST_Footprint_Lib:JST_SH_BM04B-SRSS-TB_1x04-1MP_P1.00mm_Vertical, symbol Device:LED
- added R? (x12): 330, symbol Device:R
- added R?: 50_1%, symbol Device:R
- added U? (x20): KAQY214STLD, kicad_lceda:SOP-4_L3.9-W4.4-P2.54-LS7.0-BR, symbol 0_Resistor02:KAQY214STLD
- renumbered R9 to R12, R11 to R13, R13 to R14, R17 to R16, R19 to R17, R8 to R18, R10 to R19, R12 to R20, R14 to R21, R16 to R22, R18 to R23, U7 to U11, U8 to U12, U9 to U13, U10 to U14, U11 to U15, U12 to U16
Connections:
- wire segments 17 -> 24
Other:
- moved on the sheet: R12, R13, R14, R15, R16, R17, R18, R19, R20, R21, R22, R23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
