File: Resistor_02/Resistor_02/Resistor_Network.sch (KiCad schematic (older format))
At the start: 24 parts

Commit message: Update
Parts:
- removed LED? (x6): LTST-C190GKT_LED, kicad_lceda:LED0603-RD, symbol 0_Resistor02:LTST-C190GKT_LED
- added D? (x6): LED, JST_Footprint_Lib:JST_SH_BM04B-SRSS-TB_1x04-1MP_P1.00mm_Vertical, symbol Device:LED
- gave numbers to parts that had none: 18
Connections:
- net at U7.1 (A): now also D?.1 (K)
- net at U8.1 (A): now also D?.1 (K)
- net at U9.1 (A): now also D?.1 (K)
- net at U10.1 (A): now also D?.1 (K)
- net at U12.1 (A): now also D?.1 (K)
- net at U11.1 (A): now also D?.1 (K)
- net at R9.2: now also D?.2 (A)
- net at R11.2: now also D?.2 (A)
- net at R13.2: now also D?.2 (A)
- net at R15.2: now also D?.2 (A)
- net at R17.2: now also D?.2 (A)
- net at R19.2: now also D?.2 (A)
Other:
- moved on the sheet: R11, R13, R15, R17, R19, R9

Commit message: Upddate
Parts:
- removed D? (x6): LED, JST_Footprint_Lib:JST_SH_BM04B-SRSS-TB_1x04-1MP_P1.00mm_Vertical, symbol Device:LED
- added R? (x12): 330, symbol Device:R
- added U? (x18): KAQY214STLD, kicad_lceda:SOP-4_L3.9-W4.4-P2.54-LS7.0-BR, symbol 0_Resistor02:KAQY214STLD
- renumbered R9 to R12, R11 to R13, R13 to R14, R17 to R16, R19 to R17, R8 to R18, R10 to R19, R12 to R20, R14 to R21, R16 to R22, R18 to R23, U7 to U11, U8 to U12, U9 to U13, U10 to U14, U11 to U15, U12 to U16
Connections:
- net GND: now also U?.2 (K), U?.2 (K), U?.2 (K), U?.2 (K), U?.2 (K), U?.2 (K), U?.2 (K), U?.2 (K), U?.2 (K), U?.2 (K), U?.2 (K), U?.2 (K), U?.2 (K), U?.2 (K), U?.2 (K), U?.2 (K), U?.2 (K), U?.2 (K); no longer U12.2 (K), U14.2 (K)
- net at R18.1: no longer U11.3 (S1)
- net at U12.3 (S1): no longer R19.1
- net at R20.1: no longer U13.3 (S1)
- net at U14.3 (S1): no longer R21.1
- net at U16.3 (S1): no longer R23.1
- net at R22.1: no longer U15.3 (S1)
- net Input renamed V+
- net V+: now also U?.4 (S), U?.4 (S), U?.4 (S); no longer U11.4 (S), U13.4 (S), U15.4 (S)
- removed net Output: R18.2, R19.2, R20.2, R21.2, R22.2, R23.2
- new net: R?.1, U?.1 (A) (x12)
- new net I+: U11.3 (S1), U13.3 (S1), U15.3 (S1), U?.3 (S1), U?.3 (S1), U?.3 (S1)
Other:
- moved on the sheet: R12, R18, R19, R20, R21, R22, R23, U11, U12, U13, U14, U15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

Commit message: Update
Nearly finished versions of simple and Calibrator board
Parts:
- removed R12, R13, R14, R15, R16, R17: 50_1%, symbol Device:R
- added LED? (x6): LTST-C190GKT_LED, kicad_lceda:LED0603-RD, symbol 0_Resistor02:LTST-C190GKT_LED
- added R? (x6): 330, symbol Device:R
Connections:
- net GND: no longer U11.2 (K), U13.2 (K), U15.2 (K), U16.2 (K), U?.2 (K), U?.2 (K), U?.2 (K), U?.2 (K), U?.2 (K), U?.2 (K), U?.2 (K), U?.2 (K), U?.2 (K), U?.2 (K), U?.2 (K), U?.2 (K), U?.2 (K), U?.2 (K), U?.2 (K), U?.2 (K), U?.2 (K)
- net I_04: now also U11.2 (K)
- net I_05: now also U12.2 (K), U?.2 (K), U?.2 (K)
- net I_06: now also U13.2 (K)
- net I_07: now also U14.2 (K), U?.2 (K), U?.2 (K)
- net at U11.1 (A): now also LED?.1 (-)
- net at U12.1 (A): now also R?.2
- net at U13.1 (A): now also LED?.1 (-)
- net at U14.1 (A): now also R?.2
- net at U16.1 (A): now also R?.2
- net at U15.1 (A): now also LED?.1 (-)
- net at U?.1 (A): now also R?.2 (x3)
- net at U?.1 (A): now also LED?.1 (-) (x3)
- net 3.3V: now reaches R?.2
- net 3.3V: now also LED?.2 (+), R?.1, R?.1
- new net I_10: U15.2 (K)
- new net I_11: U16.2 (K), U?.2 (K), U?.2 (K)
- new net I_12: U?.2 (K)
- new net I_13: U?.2 (K), U?.2 (K), U?.2 (K)
Other:
- moved on the sheet: R18, R19, R20, R21, R22, R23, R?, U?
