File: Calibrator_02/Calibrator_02/Calibrator_02_wResistors.sch (KiCad schematic (older format))
At the start: 22 parts, among them J1 DB9_Female_MountingHoles, J2 Conn_01x01_Female, J3 Conn_01x01_Female, J4 Conn_01x04, J5 Conn_01x04, J6 Conn_Coaxial, U1 KAQY214STLD, U10 AW9523BTQR, U2 KAQY214STLD, U3 KAQY214STLD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

Commit message: Fixed jst pinouts and made Cali board
Parts:
- removed J6: Conn_Coaxial, Connector_Coaxial:SMA_Amphenol_901-144_Vertical, symbol Connector:Conn_Coaxial
- added R1, R2, R4, R5, R7, R8: 390, Resistor_SMD:R_0603_1608Metric, symbol Device:R
- added R3, R6: 240, Resistor_SMD:R_0402_1005Metric, symbol Device:R
- JP?: renamed from JP1; footprint Jumper:SolderJumper-2_P1.3mm_Open_RoundedPad1.0x1.5mm -> (none)
Connections:
- net +3V3: now also R1.1, R2.1, R3.2, R4.1, R5.2, R6.1, R7.2, R8.2; no longer D1.2 (A), D2.2 (A), U1.1 (A), U2.1 (A), U4.1 (A), U5.1 (A), U7.1 (A), U8.1 (A)
- new net: R4.2, U4.1 (A)
- new net: R7.1, U7.1 (A)
- new net: R5.1, U5.1 (A)
- new net: R2.2, U2.1 (A)
- new net: R8.1, U8.1 (A)
- new net: R1.2, U1.1 (A)
- new net: D2.2 (A), R6.2
- new net: D1.2 (A), R3.1
Changed lines of the file:
@@
 Text Label 4500 1700 0    50   ~ 0
 I_01
+$Comp
+L Device:R R4
+U 1 1 628B5D57
+P 5100 1550
+F 0 "R4" H 5170 1596 50  0000 L CNN
+F 1 "390" H 5170 1505 50  0000 L CNN
+F 2 "Resistor_SMD:R_0603_1608Metric" V 5030 1550 50  0001 C CNN
+F 3 "~" H 5100 1550 50  0001 C CNN
+F 4 "C723655" H 5100 1550 50  0001 C CNN "LCSC"
+	1    5100 1550
+	1    0    0    -1
+$EndComp
 Text Label 5950 1600 0    50   ~ 0
 I_01
+$Comp
+L Device:R R2
+U 1 1 628B68B9
+P 6550 1450
+F 0 "R2" H 6620 1496 50  0000 L CNN
+F 1 "390" H 6620 1405 50  0000 L CNN
+F 2 "Resistor_SMD:R_0603_1608Metric" V 6480 1450 50  0001 C CNN
+F 3 "~" H 6550 1450 50  0001 C CNN
+F 4 "C723655" H 6550 1450 50  0001 C CNN "LCSC"
+	1    6550 1450
+	1    0    0    -1
+$EndComp
 Text Label 7300 1500 0    50   ~ 0
 I_01
+$Comp
+L Device:R R1
+U 1 1 628B74AE
+P 7900 1350
+F 0 "R1" H 7970 1396 50  0000 L CNN
+F 1 "390" H 7970 1305 50  0000 L CNN
+F 2 "Resistor_SMD:R_0603_1608Metric" V 7830 1350 50  0001 C CNN
+F 3 "~" H 7900 1350 50  0001 C CNN
+F 4 "C723655" H 7900 1350 50  0001 C CNN "LCSC"
+	1    7900 1350
+	1    0    0    -1
+$EndComp
 Text Label 5100 4800 3    50   ~ 0
 I_03
+$Comp
+L Device:R R7
+U 1 1 628B8C18
+P 4500 4950
+F 0 "R7" H 4570 4996 50  0000 L CNN
+F 1 "390" H 4570 4905 50  0000 L CNN
+F 2 "Resistor_SMD:R_0603_1608Metric" V 4430 4950 50  0001 C CNN
+F 3 "~" H 4500 4950 50  0001 C CNN
+F 4 "C723655" H 4500 4950 50  0001 C CNN "LCSC"
+F 5 "0603" H 4500 4950 50  0001 C CNN "Size"
+	1    4500 4950
+	1    0    0    -1
+$EndComp
 Text Label 6550 4850 3    50   ~ 0
 I_03
+$Comp
+L Device:R R8
+U 1 1 628B9EAB
+P 5950 5000
+F 0 "R8" H 6020 5046 50  0000 L CNN
+F 1 "390" H 6050 4950 50  0000 L CNN
+F 2 "Resistor_SMD:R_0603_1608Metric" V 5880 5000 50  0001 C CNN
+F 3 "~" H 5950 5000 50  0001 C CNN
+F 4 "C723655" H 5950 5000 50  0001 C CNN "LCSC"
+	1    5950 5000
+	1    0    0    -1
+$EndComp
 Text Label 7900 4750 3    50   ~ 0
 I_03
+$Comp
+L Device:R R5
+U 1 1 628BA99D
+P 7300 4900
+F 0 "R5" H 7370 4946 50  0000 L CNN
+F 1 "390" H 7370 4855 50  0000 L CNN
+F 2 "Resistor_SMD:R_0603_1608Metric" V 7230 4900 50  0001 C CNN
+F 3 "~" H 7300 4900 50  0001 C CNN
+F 4 "C723655" H 7300 4900 50  0001 C CNN "LCSC"
+	1    7300 4900
+	1    0    0    -1
+$EndComp
 $Comp
 L power:GNDS #PWR0101
@@
 	-1   0    0    1
 $EndComp
+$Comp
+L Device:R R6
+U 1 1 62885109
+P 3700 1150
+F 0 "R6" H 3770 1196 50  0000 L CNN
+F 1 "240" H 3770 1105 50  0000 L CNN
+F 2 "Resistor_SMD:R_0402_1005Metric" V 3630 1150 50  0001 C CNN
+F 3 "" H 3700 1150 50  0001 C CNN
+F 4 "C470040" H 3700 1150 50  0001 C CNN "LCSC"
+F 5 "R0402" H 3700 1150 50  0001 C CNN "Size"
+	1    3700 1150
+	1    0    0    -1
+$EndComp
+Wire Wire Line
+	3700 700  3700 1000
+Wire Wire Line
+	5100 700  5100 1400
+Wire Wire Line
+	6550 700  6550 1300
+Wire Wire Line
+	7900 700  7900 1200
+Wire Wire Line
+	2100 5500 3100 5500
+$Comp
+L Device:R R3
+U 1 1 62892A48
+P 3100 5350
+F 0 "R3" H 3170 5396 50  0000 L CNN
+F 1 "240" H 3170 5305 50  0000 L CNN
+F 2 "Resistor_SMD:R_0402_1005Metric" V 3030 5350 50  0001 C CNN
+F 3 "" H 3100 5350 50  0001 C CNN
+F 4 "C470040" H 3100 5350 50  0001 C CNN "LCSC"
+F 5 "R0402" H 3100 5350 50  0001 C CNN "Size"
+	1    3100 5350
+	1    0    0    -1
+$EndComp
+Wire Wire Line
+	7300 5050 7300 5500
+Connection ~ 3100 5500
+Wire Wire Line
+	4500 5100 4500 5500
+Wire Wire Line
+	3100 5500 4500 5500
 Connection ~ 4500 5500
 Wire Wire Line
 	4500 5500 5950 5500
+Wire Wire Line
+	5950 5150 5950 5500
 Connection ~ 5950 5500
 Wire Wire Line
@@
 $EndComp
 Wire Wire Line
+	3700 1300 3700 1350
+Wire Wire Line
 	3700 1700 3700 1650
 $Comp
@@
 	0    1    1    0
 $EndComp
+Wire Wire Line
+	3100 5200 3100 5100
 Text Notes 850  6600 2    50   ~ 0
 Gnd\n
@@
 	8350 2900 9050 2900
 Wire Wire Line
-	8450 3000 8650 3000
+	8450 3000 8950 3000
 Wire Wire Line
 	8950 2500 8950 3000
@@
 	1700 6500 1800 6500
 $Comp
-L Device:Jumper JP1
+L Device:Jumper JP?
 U 1 1 627E9ED5
 P 1800 6200
-F 0 "JP1" V 1754 6327 50  0000 L CNN
+F 0 "JP?" V 1754 6327 50  0000 L CNN
 F 1 "Jumper" V 1845 6327 50  0000 L CNN
-F 2 "Jumper:SolderJumper-2_P1.3mm_Open_RoundedPad1.0x1.5mm" H 1800 6200 50  0001 C CNN
+F 2 "" H 1800 6200 50  0001 C CNN
 F 3 "~" H 1800 6200 50  0001 C CNN
 	1    1800 6200
@@
 	1800 6500 2750 6500
 $Comp
-L power:+3.3V #PWR0107
+L power:+3.3V #PWR?
 U 1 1 627EAC45
 P 1800 5900
-F 0 "#PWR0107" H 1800 5750 50  0001 C CNN
+F 0 "#PWR?" H 1800 5750 50  0001 C CNN
 F 1 "+3.3V" H 1815 6073 50  0000 C CNN
 F 2 "" H 1800 5900 50  0001 C CNN
@@
 	1    0    0    -1
 $EndComp
-Wire Wire Line
-	7300 4750 7300 5500
-Wire Wire Line
-	5950 4850 5950 5500
-Wire Wire Line
-	4500 4800 4500 5500
-Wire Wire Line
-	2100 5500 3100 5500
-Wire Wire Line
-	3100 5100 3100 5500
-Connection ~ 3100 5500
-Wire Wire Line
-	3100 5500 4500 5500
-Wire Wire Line
-	7900 700  7900 1500
-Wire Wire Line
-	6550 700  6550 1600
-Wire Wire Line
-	5100 700  5100 1700
-Wire Wire Line
-	3700 700  3700 1350
-$Comp
-L Connector:Conn_Coaxial J?
-U 1 1 628F1540
-P 8650 3400
-AR Path="/6283D226/628F1540" Ref="J?"  Part="1"
-AR Path="/628F1540" Ref="J6"  Part="1"
-F 0 "J6" H 8750 3375 50  0000 L CNN
-F 1 "Conn_Coaxial" H 8750 3284 50  0000 L CNN
-F 2 "Connector_Coaxial:SMA_Amphenol_901-144_Vertical" H 8650 3400 50  0001 C CNN
-F 3 " ~" H 8650 3400 50  0001 C CNN
-	1    8650 3400
-	-1   0    0    1
-$EndComp
-Wire Wire Line
-	8850 2800 8850 3400
-Wire Wire Line
-	8650 3000 8650 3200
-Connection ~ 8650 3000
-Wire Wire Line
-	8650 3000 8950 3000
 $EndSCHEMATC
