File: Calibrator_02/Calibrator_02/Calibrator_02.sch (KiCad schematic (older format))
At the start: 28 parts, among them J1 DB9_Female_MountingHoles, J2 Conn_01x01_Female, U1 KAQY214STLD, U2 KAQY214STLD, U3 KAQY214STLD, U4 KAQY214STLD, U5 KAQY214STLD, U6 KAQY214STLD, U7 KAQY214STLD, U8 KAQY214STLD, U9 A1001WR-S-04PD01

Commit message: Update
Nearly finished versions of simple and Calibrator board
Parts:
- removed LED? (x2): LTST-C190GKT_LED, kicad_lceda:LED0603-RD, symbol 0_Resistor02:LTST-C190GKT_LED
- removed U9: A1001WR-S-04PD01, JST_Footprint_Lib:JST_SH_BM04B-SRSS-TB_1x04-1MP_P1.00mm_Vertical, symbol 0_Resistor02:A1001WR-S-04PD01
- added D1, D2: LED, 0_Resistor_02:LED0603-RD, symbol Device:LED
- added J4, J5: Conn_01x04, Connector_JST:JST_SH_SM04B-SRSS-TB_1x04-1MP_P1.00mm_Horizontal, symbol Connector_Generic:Conn_01x04
- C1: renamed from 1uF; value C -> 1uF; footprint (none) -> Capacitor_SMD:C_0402_1005Metric; Footprint size  0603 -> 0402; LCSC C1656 -> C77009
- J1: footprint (none) -> 0_Resistor_02:DSUB-TH_DMR-9S; LCSC (none) -> C141882
- J2: footprint (none) -> Connector_PinSocket_2.54mm:PinSocket_1x01_P2.54mm_Horizontal
- J3: renamed from J?; footprint (none) -> Connector_PinSocket_2.54mm:PinSocket_1x01_P2.54mm_Horizontal
- R1, R2, R4, R5, R7, R8: footprint (none) -> Resistor_SMD:R_0603_1608Metric
- R23, R40, R41, R42: renamed from 4.7K; value R -> 4.7K; footprint (none) -> Resistor_SMD:R_0805_2012Metric
- R3, R6: renamed from R?; footprint (none) -> Resistor_SMD:R_0402_1005Metric
- U1, U2, U3, U4, U5, U6, U7, U8: footprint kicad_lceda:SOP-4_L3.9-W4.4-P2.54-LS7.0-BR -> 0_Resistor_02:SOP-4_L3.9-W4.4-P2.54-LS7.0-BR
- U10: renamed from U?; footprint kicad_lceda:TQFN-24_L4.0-W4.0-P0.50-TL-EP -> 0_Resistor_02:TQFN-24_L4.0-W4.0-P0.50-TL-EP
Connections:
- wire segments 66 -> 94
Other:
- note added: "Gnd\n"
- note added: "scl"
- note added: "sda"
- note added: "vcc\n"
- moved on the sheet: R41

Commit message: Fixed jst pinouts and made Cali board
Parts:
- removed R1, R2, R4, R5, R7, R8: 390, Resistor_SMD:R_0603_1608Metric, symbol Device:R
- removed R3, R6: 240, Resistor_SMD:R_0402_1005Metric, symbol Device:R
- removed R40: 4.7K, Resistor_SMD:R_0805_2012Metric, symbol Device:R
- added J6: Conn_Coaxial, Connector_Coaxial:SMA_Amphenol_901-144_Vertical, symbol Connector:Conn_Coaxial
- added JP1: Jumper, Jumper:SolderJumper-2_P1.3mm_Open_RoundedPad1.0x1.5mm, symbol Device:Jumper
Connections:
- net +3V3: now also D1.2 (A), D2.2 (A), U1.1 (A), U2.1 (A), U4.1 (A), U5.1 (A), U7.1 (A), U8.1 (A), JP1.1
- net GND: now also J1.3
- net GNDS: no longer J1.3
- net Resistor_Network/I-: now also J4.4 (Pin_4); no longer J4.3 (Pin_3)
- net Resistor_Network/V+: now also J6.1 (In)
- net Resistor_Network/V-: now also J4.3 (Pin_3), J6.2 (Ext); no longer J4.4 (Pin_4)
- net at J3.1 (Pin_1), U10.23 (RSTN): now also JP1.2
Changed lines of the file:
@@
 Text Label 4500 1700 0    50   ~ 0
 I_01
-$Comp
-L Device:R R4
-U 1 1 628B5D57
-P 5100 1550
-F 0 "R4" H 5170 1596 50  0000 L CNN
-F 1 "390" H 5170 1505 50  0000 L CNN
-F 2 "Resistor_SMD:R_0603_1608Metric" V 5030 1550 50  0001 C CNN
-F 3 "~" H 5100 1550 50  0001 C CNN
-F 4 "C723655" H 5100 1550 50  0001 C CNN "LCSC"
-	1    5100 1550
-	1    0    0    -1
-$EndComp
 Text Label 5950 1600 0    50   ~ 0
 I_01
-$Comp
-L Device:R R2
-U 1 1 628B68B9
-P 6550 1450
-F 0 "R2" H 6620 1496 50  0000 L CNN
-F 1 "390" H 6620 1405 50  0000 L CNN
-F 2 "Resistor_SMD:R_0603_1608Metric" V 6480 1450 50  0001 C CNN
-F 3 "~" H 6550 1450 50  0001 C CNN
-F 4 "C723655" H 6550 1450 50  0001 C CNN "LCSC"
-	1    6550 1450
-	1    0    0    -1
-$EndComp
 Text Label 7300 1500 0    50   ~ 0
 I_01
-$Comp
-L Device:R R1
-U 1 1 628B74AE
-P 7900 1350
-F 0 "R1" H 7970 1396 50  0000 L CNN
-F 1 "390" H 7970 1305 50  0000 L CNN
-F 2 "Resistor_SMD:R_0603_1608Metric" V 7830 1350 50  0001 C CNN
-F 3 "~" H 7900 1350 50  0001 C CNN
-F 4 "C723655" H 7900 1350 50  0001 C CNN "LCSC"
-	1    7900 1350
-	1    0    0    -1
-$EndComp
 Text Label 5100 4800 3    50   ~ 0
 I_03
-$Comp
-L Device:R R7
-U 1 1 628B8C18
-P 4500 4950
-F 0 "R7" H 4570 4996 50  0000 L CNN
-F 1 "390" H 4570 4905 50  0000 L CNN
-F 2 "Resistor_SMD:R_0603_1608Metric" V 4430 4950 50  0001 C CNN
-F 3 "~" H 4500 4950 50  0001 C CNN
-F 4 "C723655" H 4500 4950 50  0001 C CNN "LCSC"
-F 5 "0603" H 4500 4950 50  0001 C CNN "Size"
-	1    4500 4950
-	1    0    0    -1
-$EndComp
 Text Label 6550 4850 3    50   ~ 0
 I_03
-$Comp
-L Device:R R8
-U 1 1 628B9EAB
-P 5950 5000
-F 0 "R8" H 6020 5046 50  0000 L CNN
-F 1 "390" H 6050 4950 50  0000 L CNN
-F 2 "Resistor_SMD:R_0603_1608Metric" V 5880 5000 50  0001 C CNN
-F 3 "~" H 5950 5000 50  0001 C CNN
-F 4 "C723655" H 5950 5000 50  0001 C CNN "LCSC"
-	1    5950 5000
-	1    0    0    -1
-$EndComp
 Text Label 7900 4750 3    50   ~ 0
 I_03
-$Comp
-L Device:R R5
-U 1 1 628BA99D
-P 7300 4900
-F 0 "R5" H 7370 4946 50  0000 L CNN
-F 1 "390" H 7370 4855 50  0000 L CNN
-F 2 "Resistor_SMD:R_0603_1608Metric" V 7230 4900 50  0001 C CNN
-F 3 "~" H 7300 4900 50  0001 C CNN
-F 4 "C723655" H 7300 4900 50  0001 C CNN "LCSC"
-	1    7300 4900
-	1    0    0    -1
-$EndComp
-$Comp
-L power:GNDS #PWR0101
-U 1 1 6299368D
-P 2350 3200
-F 0 "#PWR0101" H 2350 2950 50  0001 C CNN
-F 1 "GNDS" V 2355 3072 50  0000 R CNN
-F 2 "" H 2350 3200 50  0001 C CNN
-F 3 "" H 2350 3200 50  0001 C CNN
-	1    2350 3200
-	0    -1   -1   0
-$EndComp
 Wire Wire Line
 	2200 3200 2350 3200
@@
 Wire Wire Line
 	8350 3250 8350 2900
-Wire Wire Line
-	8350 2900 8950 2900
 Connection ~ 6550 3250
 Wire Wire Line
@@
 Wire Wire Line
 	8450 3300 8450 3000
-Wire Wire Line
-	8450 3000 9050 3000
 Connection ~ 7900 3300
 Wire Wire Line
@@
 $EndComp
 $Comp
-L power:+3.3V #PWR0107
-U 1 1 6281DAD4
-P 1800 5900
-F 0 "#PWR0107" H 1800 5750 50  0001 C CNN
-F 1 "+3.3V" H 1815 6073 50  0000 C CNN
-F 2 "" H 1800 5900 50  0001 C CNN
-F 3 "" H 1800 5900 50  0001 C CNN
-	1    1800 5900
-	-1   0    0    -1
-$EndComp
-Wire Wire Line
-	1700 6500 1800 6500
-Wire Wire Line
-	1800 6500 1800 6200
-Connection ~ 1800 6500
-$Comp
-L Device:R R40
-U 1 1 6281DADF
-P 1800 6050
-F 0 "R40" H 1870 6096 50  0000 L CNN
-F 1 "4.7K" H 1870 6005 50  0000 L CNN
-F 2 "Resistor_SMD:R_0805_2012Metric" V 1730 6050 50  0001 C CNN
-F 3 "~" H 1800 6050 50  0001 C CNN
-F 4 "C17673" H 1800 6050 50  0001 C CNN "LCSC"
-F 5 "0805" H 1800 6050 50  0001 C CNN "FT size"
-	1    1800 6050
-	1    0    0    -1
-$EndComp
-Wire Wire Line
-	1800 6500 2750 6500
-$Comp
 L Device:C C1
 U 1 1 62823101
@@
 	-1   0    0    1
 $EndComp
-$Comp
-L Device:R R6
-U 1 1 62885109
-P 3700 1150
-F 0 "R6" H 3770 1196 50  0000 L CNN
-F 1 "240" H 3770 1105 50  0000 L CNN
-F 2 "Resistor_SMD:R_0402_1005Metric" V 3630 1150 50  0001 C CNN
-F 3 "" H 3700 1150 50  0001 C CNN
-F 4 "C470040" H 3700 1150 50  0001 C CNN "LCSC"
-F 5 "R0402" H 3700 1150 50  0001 C CNN "Size"
-	1    3700 1150
-	1    0    0    -1
-$EndComp
-Wire Wire Line
-	3700 700  3700 1000
-Wire Wire Line
-	5100 700  5100 1400
-Wire Wire Line
-	6550 700  6550 1300
-Wire Wire Line
-	7900 700  7900 1200
-Wire Wire Line
-	2100 5500 3100 5500
-$Comp
-L Device:R R3
-U 1 1 62892A48
-P 3100 5350
-F 0 "R3" H 3170 5396 50  0000 L CNN
-F 1 "240" H 3170 5305 50  0000 L CNN
-F 2 "Resistor_SMD:R_0402_1005Metric" V 3030 5350 50  0001 C CNN
-F 3 "" H 3100 5350 50  0001 C CNN
-F 4 "C470040" H 3100 5350 50  0001 C CNN "LCSC"
-F 5 "R0402" H 3100 5350 50  0001 C CNN "Size"
-	1    3100 5350
-	1    0    0    -1
-$EndComp
-Wire Wire Line
-	7300 5050 7300 5500
-Connection ~ 3100 5500
-Wire Wire Line
-	4500 5100 4500 5500
-Wire Wire Line
-	3100 5500 4500 5500
 Connection ~ 4500 5500
 Wire Wire Line
 	4500 5500 5950 5500
-Wire Wire Line
-	5950 5150 5950 5500
 Connection ~ 5950 5500
 Wire Wire Line
@@
 Wire Wire Line
 	8850 2800 9350 2800
-Wire Wire Line
-	8950 2500 8950 2900
-Connection ~ 8950 2900
-Wire Wire Line
-	8950 2900 9350 2900
-Wire Wire Line
-	9050 2500 9050 3000
-Connection ~ 9050 3000
-Wire Wire Line
-	9050 3000 9350 3000
 $Comp
 L power:+3.3V #PWR01
@@
 $EndComp
 Wire Wire Line
-	3700 1300 3700 1350
-Wire Wire Line
 	3700 1700 3700 1650
 $Comp
@@
 	0    1    1    0
 $EndComp
-Wire Wire Line
-	3100 5200 3100 5100
 Text Notes 850  6600 2    50   ~ 0
 Gnd\n
@@
 Wire Wire Line
 	1150 6350 1150 6600
+Wire Wire Line
+	8350 2900 9050 2900
+Wire Wire Line
+	8450 3000 8650 3000
+Wire Wire Line
+	8950 2500 8950 3000
+Connection ~ 8950 3000
+Wire Wire Line
+	8950 3000 9350 3000
+Wire Wire Line
+	9050 2500 9050 2900
+Connection ~ 9050 2900
+Wire Wire Line
+	9050 2900 9350 2900
+Wire Wire Line
+	1700 6500 1800 6500
+$Comp
+L Device:Jumper JP1
+U 1 1 627E9ED5
+P 1800 6200
+F 0 "JP1" V 1754 6327 50  0000 L CNN
+F 1 "Jumper" V 1845 6327 50  0000 L CNN
+F 2 "Jumper:SolderJumper-2_P1.3mm_Open_RoundedPad1.0x1.5mm" H 1800 6200 50  0001 C CNN
+F 3 "~" H 1800 6200 50  0001 C CNN
+	1    1800 6200
+	0    1    1    0
+$EndComp
+Connection ~ 1800 6500
+Wire Wire Line
+	1800 6500 2750 6500
+$Comp
+L power:+3.3V #PWR0107
+U 1 1 627EAC45
+P 1800 5900
+F 0 "#PWR0107" H 1800 5750 50  0001 C CNN
+F 1 "+3.3V" H 1815 6073 50  0000 C CNN
+F 2 "" H 1800 5900 50  0001 C CNN
+F 3 "" H 1800 5900 50  0001 C CNN
+	1    1800 5900
+	1    0    0    -1
+$EndComp
+Wire Wire Line
+	7300 4750 7300 5500
+Wire Wire Line
+	5950 4850 5950 5500
+Wire Wire Line
+	4500 4800 4500 5500
+Wire Wire Line
+	2100 5500 3100 5500
+Wire Wire Line
+	3100 5100 3100 5500
+Connection ~ 3100 5500
+Wire Wire Line
+	3100 5500 4500 5500
+Wire Wire Line
+	7900 700  7900 1500
+Wire Wire Line
+	6550 700  6550 1600
+Wire Wire Line
+	5100 700  5100 1700
+Wire Wire Line
+	3700 700  3700 1350
+$Comp
+L Connector:Conn_Coaxial J?
+U 1 1 628F1540
+P 8650 3400
+AR Path="/6283D226/628F1540" Ref="J?"  Part="1"
+AR Path="/628F1540" Ref="J6"  Part="1"
+F 0 "J6" H 8750 3375 50  0000 L CNN
+F 1 "Conn_Coaxial" H 8750 3284 50  0000 L CNN
+F 2 "Connector_Coaxial:SMA_Amphenol_901-144_Vertical" H 8650 3400 50  0001 C CNN
+F 3 " ~" H 8650 3400 50  0001 C CNN
+	1    8650 3400
+	-1   0    0    1
+$EndComp
+Wire Wire Line
+	8850 2800 8850 3400
+Wire Wire Line
+	8650 3000 8650 3200
+Connection ~ 8650 3000
+Wire Wire Line
+	8650 3000 8950 3000
+$Comp
+L power:GND #PWR?
+U 1 1 62A1E2CA
+P 2350 3200
+F 0 "#PWR?" H 2350 2950 50  0001 C CNN
+F 1 "GND" V 2355 3072 50  0000 R CNN
+F 2 "" H 2350 3200 50  0001 C CNN
+F 3 "" H 2350 3200 50  0001 C CNN
+	1    2350 3200
+	0    -1   -1   0
+$EndComp
 $EndSCHEMATC

Commit message: Update
Parts:
- renumbered D2 to D1, D1 to D2, J4 to J1, J1 to J2, J6 to J3, J3 to J4, J2 to J5, J5 to J6, U10 to M1, R42 to R1, R41 to R2, R23 to R3
Changed lines of the file:
@@
 	1350 6700 1150 6700
 $Comp
-L power:+3.3V #PWR021
+L power:+3.3V #PWR017
 U 1 1 6274D25F
 P 1500 7350
-F 0 "#PWR021" H 1500 7200 50  0001 C CNN
+F 0 "#PWR017" H 1500 7200 50  0001 C CNN
 F 1 "+3.3V" H 1515 7523 50  0000 C CNN
 F 2 "" H 1500 7350 50  0001 C CNN
@@
 $EndComp
 $Comp
-L power:+3.3V #PWR018
+L power:+3.3V #PWR016
 U 1 1 6274DA20
 P 1850 7200
-F 0 "#PWR018" H 1850 7050 50  0001 C CNN
+F 0 "#PWR016" H 1850 7050 50  0001 C CNN
 F 1 "+3.3V" H 1865 7373 50  0000 C CNN
 F 2 "" H 1850 7200 50  0001 C CNN
@@
 $EndComp
 $Comp
-L power:GND #PWR020
+L power:GND #PWR011
 U 1 1 6274F916
 P 2750 6300
-F 0 "#PWR020" H 2750 6050 50  0001 C CNN
+F 0 "#PWR011" H 2750 6050 50  0001 C CNN
 F 1 "GND" V 2755 6172 50  0000 R CNN
 F 2 "" H 2750 6300 50  0001 C CNN
@@
 $EndComp
 $Comp
-L Connector:DB9_Female_MountingHoles J1
+L Connector:DB9_Female_MountingHoles J2
 U 1 1 6276A70E
 P 1900 3200
-F 0 "J1" H 1818 3892 50  0000 C CNN
+F 0 "J2" H 1818 3892 50  0000 C CNN
 F 1 "DB9_Female_MountingHoles" H 1818 3801 50  0000 C CNN
 F 2 "0_Resistor_02:DSUB-TH_DMR-9S" H 1900 3200 50  0001 C CNN
@@
 Connection ~ 1350 6700
 $Comp
-L power:GND #PWR014
+L power:GND #PWR012
 U 1 1 627ED8FC
 P 1150 6350
-F 0 "#PWR014" H 1150 6100 50  0001 C CNN
+F 0 "#PWR012" H 1150 6100 50  0001 C CNN
 F 1 "GND" H 1155 6177 50  0000 C CNN
 F 2 "" H 1150 6350 50  0001 C CNN
@@
 $EndComp
 $Comp
-L power:GNDS #PWR06
+L power:GNDS #PWR04
 U 1 1 627EED50
 P 1900 3800
-F 0 "#PWR06" H 1900 3550 50  0001 C CNN
+F 0 "#PWR04" H 1900 3550 50  0001 C CNN
 F 1 "GNDS" H 1905 3627 50  0000 C CNN
 F 2 "" H 1900 3800 50  0001 C CNN
@@
 $EndComp
 $Comp
-L Connector:Conn_01x01_Female J2
+L Connector:Conn_01x01_Female J5
 U 1 1 627F98CB
 P 1850 6600
-F 0 "J2" H 1800 6750 50  0000 C CNN
+F 0 "J5" H 1800 6750 50  0000 C CNN
 F 1 "Conn_01x01_Female" H 1800 6550 50  0000 C CNN
 F 2 "Connector_PinSocket_2.54mm:PinSocket_1x01_P2.54mm_Horizontal" H 1850 6600 50  0001 C CNN
@@
 I_01
 $Comp
-L power:+3.3V #PWR019
+L power:+3.3V #PWR010
 U 1 1 6283A97E
 P 2150 6000
-F 0 "#PWR019" H 2150 5850 50  0001 C CNN
+F 0 "#PWR010" H 2150 5850 50  0001 C CNN
 F 1 "+3.3V" H 2165 6173 50  0000 C CNN
 F 2 "" H 2150 6000 50  0001 C CNN
@@
 I_07
 $Comp
-L power:+3.3V #PWR022
+L power:+3.3V #PWR019
 U 1 1 628DDA57
 P 750 7600
-F 0 "#PWR022" H 750 7450 50  0001 C CNN
+F 0 "#PWR019" H 750 7450 50  0001 C CNN
 F 1 "+3.3V" H 765 7773 50  0000 C CNN
 F 2 "" H 750 7600 50  0001 C CNN
@@
 $EndComp
 $Comp
-L power:GND #PWR08
+L power:GND #PWR06
 U 1 1 628586D7
 P 7950 4250
-F 0 "#PWR08" H 7950 4000 50  0001 C CNN
+F 0 "#PWR06" H 7950 4000 50  0001 C CNN
 F 1 "GND" H 7955 4077 50  0000 C CNN
 F 2 "" H 7950 4250 50  0001 C CNN
@@
 $EndComp
 $Comp
-L power:GND #PWR07
+L power:GND #PWR05
 U 1 1 6285CC89
 P 6550 4100
-F 0 "#PWR07" H 6550 3850 50  0001 C CNN
+F 0 "#PWR05" H 6550 3850 50  0001 C CNN
 F 1 "GND" H 6555 3927 50  0000 C CNN
 F 2 "" H 6550 4100 50  0001 C CNN
@@
 	7900 3300 7900 3650
 $Comp
-L 0_Resistor02:AW9523BTQR U10
+L 0_Resistor02:AW9523BTQR M1
 U 1 1 627BA299
 P 3500 6650
-F 0 "U10" V 3650 6650 50  0000 L CNN
+F 0 "M1" V 3650 6650 50  0000 L CNN
 F 1 "AW9523BTQR" V 3500 6500 50  0000 L CNN
 F 2 "0_Resistor_02:TQFN-24_L4.0-W4.0-P0.50-TL-EP" H 3500 7323 50  0001 C CNN
@@
 $EndComp
 $Comp
-L power:GND #PWR0102
+L power:GND #PWR014
 U 1 1 627BCD14
 P 4250 6600
-F 0 "#PWR0102" H 4250 6350 50  0001 C CNN
+F 0 "#PWR014" H 4250 6350 50  0001 C CNN
 F 1 "GND" V 4255 6472 50  0000 R CNN
 F 2 "" H 4250 6600 50  0001 C CNN
@@
 	3700 700  5100 700
 $Comp
-L power:+3.3V #PWR0103
+L power:+3.3V #PWR01
 U 1 1 6280D88E
 P 1700 700
-F 0 "#PWR0103" H 1700 550 50  0001 C CNN
+F 0 "#PWR01" H 1700 550 50  0001 C CNN
 F 1 "+3.3V" H 1715 873 50  0000 C CNN
 F 2 "" H 1700 700 50  0001 C CNN
@@
 	1650 5500 2100 5500
 $Comp
-L power:+3.3V #PWR0104
+L power:+3.3V #PWR08
 U 1 1 62812E5B
 P 1650 5500
-F 0 "#PWR0104" H 1650 5350 50  0001 C CNN
+F 0 "#PWR08" H 1650 5350 50  0001 C CNN
 F 1 "+3.3V" H 1665 5673 50  0000 C CNN
 F 2 "" H 1650 5500 50  0001 C CNN
@@
 $EndComp
 $Comp
-L Device:R R42
+L Device:R R1
 U 1 1 6281583F
 P 2150 6150
-F 0 "R42" H 2220 6196 50  0000 L CNN
+F 0 "R1" H 2220 6196 50  0000 L CNN
 F 1 "4.7K" H 2220 6105 50  0000 L CNN
 F 2 "Resistor_SMD:R_0805_2012Metric" V 2080 6150 50  0001 C CNN
@@
 $EndComp
 $Comp
-L Device:R R23
+L Device:R R3
 U 1 1 628173F4
 P 1500 7200
-F 0 "R23" H 1570 7246 50  0000 L CNN
+F 0 "R3" H 1570 7246 50  0000 L CNN
 F 1 "4.7K" H 1570 7155 50  0000 L CNN
 F 2 "Resistor_SMD:R_0805_2012Metric" V 1430 7200 50  0001 C CNN
@@
 $EndComp
 $Comp
-L Device:R R41
+L Device:R R2
 U 1 1 6281855E
 P 1850 7050
-F 0 "R41" H 1920 7096 50  0000 L CNN
+F 0 "R2" H 1920 7096 50  0000 L CNN
 F 1 "4.7K" H 1920 7005 50  0000 L CNN
 F 2 "Resistor_SMD:R_0805_2012Metric" V 1780 7050 50  0001 C CNN
@@
 $EndComp
 $Comp
-L power:+3.3V #PWR0105
-U 1 1 6281A8FB
-P 2750 6400
-F 0 "#PWR0105" H 2750 6250 50  0001 C CNN
-F 1 "+3.3V" V 2765 6528 50  0000 L CNN
-F 2 "" H 2750 6400 50  0001 C CNN
-F 3 "" H 2750 6400 50  0001 C CNN
-	1    2750 6400
-	0    -1   -1   0
-$EndComp
-$Comp
-L power:+3.3V #PWR0106
-U 1 1 6281B1AA
-P 3250 7400
-F 0 "#PWR0106" H 3250 7250 50  0001 C CNN
-F 1 "+3.3V" H 3265 7573 50  0000 C CNN
-F 2 "" H 3250 7400 50  0001 C CNN
-F 3 "" H 3250 7400 50  0001 C CNN
-	1    3250 7400
-	-1   0    0    1
-$EndComp
-$Comp
-L Connector:Conn_01x01_Female J3
+L Connector:Conn_01x01_Female J4
 U 1 1 6281DACE
 P 1500 6500
-F 0 "J3" H 1450 6650 50  0000 C CNN
+F 0 "J4" H 1450 6650 50  0000 C CNN
 F 1 "Conn_01x01_Female" H 1400 6600 50  0000 C CNN
 F 2 "Connector_PinSocket_2.54mm:PinSocket_1x01_P2.54mm_Horizontal" H 1500 6500 50  0001 C CNN
@@
 Connection ~ 2100 5500
 $Comp
-L power:GND #PWR0108
+L power:GND #PWR07
 U 1 1 6282423C
 P 2100 5200
-F 0 "#PWR0108" H 2100 4950 50  0001 C CNN
+F 0 "#PWR07" H 2100 4950 50  0001 C CNN
 F 1 "GND" H 2105 5027 50  0000 C CNN
 F 2 "" H 2100 5200 50  0001 C CNN
@@
 	5950 5500 7300 5500
 $Comp
-L Connector_Generic:Conn_01x04 J4
+L Connector_Generic:Conn_01x04 J1
 U 1 1 627E1405
 P 8850 2300
-F 0 "J4" V 8814 2012 50  0000 R CNN
+F 0 "J1" V 8814 2012 50  0000 R CNN
 F 1 "Conn_01x04" V 8723 2012 50  0000 R CNN
 F 2 "Connector_JST:JST_SH_SM04B-SRSS-TB_1x04-1MP_P1.00mm_Horizontal" H 8850 2300 50  0001 C CNN
@@
 	8850 2800 9350 2800
 $Comp
-L power:+3.3V #PWR01
+L power:+3.3V #PWR02
 U 1 1 629288EE
 P 10450 2800
-F 0 "#PWR01" H 10450 2650 50  0001 C CNN
+F 0 "#PWR02" H 10450 2650 50  0001 C CNN
 F 1 "+3.3V" V 10465 2928 50  0000 L CNN
 F 2 "" H 10450 2800 50  0001 C CNN
@@
 I_17
 $Comp
-L Device:LED D2
+L Device:LED D1
 U 1 1 629325F5
 P 3700 1500
-F 0 "D2" V 3739 1382 50  0000 R CNN
+F 0 "D1" V 3739 1382 50  0000 R CNN
 F 1 "LED" V 3648 1382 50  0000 R CNN
 F 2 "0_Resistor_02:LED0603-RD" H 3700 1500 50  0001 C CNN
@@
 	3700 1700 3700 1650
 $Comp
-L Device:LED D1
+L Device:LED D2
 U 1 1 62937D23
 P 3100 4950
-F 0 "D1" H 3093 5167 50  0000 C CNN
+F 0 "D2" H 3093 5167 50  0000 C CNN
 F 1 "LED" H 3093 5076 50  0000 C CNN
 F 2 "0_Resistor_02:LED0603-RD" H 3100 4950 50  0001 C CNN
@@
 	3100 1650 3100 1700
 $Comp
-L Connector_Generic:Conn_01x04 J5
+L Connector_Generic:Conn_01x04 J6
 U 1 1 62A90CC6
 P 950 6700
-F 0 "J5" H 868 7017 50  0000 C CNN
+F 0 "J6" H 868 7017 50  0000 C CNN
 F 1 "Conn_01x04" H 868 6926 50  0000 C CNN
 F 2 "Connector_JST:JST_SH_SM04B-SRSS-TB_1x04-1MP_P1.00mm_Horizontal" H 950 6700 50  0001 C CNN
@@
 	1800 6500 2750 6500
 $Comp
-L power:+3.3V #PWR0107
+L power:+3.3V #PWR09
 U 1 1 627EAC45
 P 1800 5900
-F 0 "#PWR0107" H 1800 5750 50  0001 C CNN
+F 0 "#PWR09" H 1800 5750 50  0001 C CNN
 F 1 "+3.3V" H 1815 6073 50  0000 C CNN
 F 2 "" H 1800 5900 50  0001 C CNN
@@
 P 8650 3400
 AR Path="/6283D226/628F1540" Ref="J?"  Part="1"
-AR Path="/628F1540" Ref="J6"  Part="1"
-F 0 "J6" H 8750 3375 50  0000 L CNN
+AR Path="/628F1540" Ref="J3"  Part="1"
+F 0 "J3" H 8750 3375 50  0000 L CNN
 F 1 "Conn_Coaxial" H 8750 3284 50  0000 L CNN
 F 2 "Connector_Coaxial:SMA_Amphenol_901-144_Vertical" H 8650 3400 50  0001 C CNN
@@
 	8650 3000 8950 3000
 $Comp
-L power:GND #PWR?
+L power:GND #PWR03
 U 1 1 62A1E2CA
 P 2350 3200
-F 0 "#PWR?" H 2350 2950 50  0001 C CNN
+F 0 "#PWR03" H 2350 2950 50  0001 C CNN
 F 1 "GND" V 2355 3072 50  0000 R CNN
 F 2 "" H 2350 3200 50  0001 C CNN
@@
 	0    -1   -1   0
 $EndComp
+$Comp
+L power:+3.3V #PWR013
+U 1 1 6281A8FB
+P 2750 6400
+F 0 "#PWR013" H 2750 6250 50  0001 C CNN
+F 1 "+3.3V" V 2765 6528 50  0000 L CNN
+F 2 "" H 2750 6400 50  0001 C CNN
+F 3 "" H 2750 6400 50  0001 C CNN
+	1    2750 6400
+	0    -1   -1   0
+$EndComp
+$Comp
+L power:+3.3V #PWR018
+U 1 1 6281B1AA
+P 3250 7400
+F 0 "#PWR018" H 3250 7250 50  0001 C CNN
+F 1 "+3.3V" H 3400 7650 50  0000 C CNN
+F 2 "" H 3250 7400 50  0001 C CNN
+F 3 "" H 3250 7400 50  0001 C CNN
+	1    3250 7400
+	-1   0    0    1
+$EndComp
 $EndSCHEMATC
