File: Calibrator_02/Calibrator_02/Calibrator_02_wResistors.kicad_pcb (KiCad board)
At the start: 2 copper layers, 100 x 50 mm, 88 parts, among them J1 Conn_01x04, J2 DB9_Female_MountingHoles, J3 Conn_Coaxial, J5 Conn_01x01_Female, J6 Conn_01x04, M1 AW9523BTQR, U1 KAQY214STLD, U10 KAQY214STLD, U11 KAQY214STLD, U12 KAQY214STLD, U13 KAQY214STLD, U14 KAQY214STLD, U15 KAQY214STLD, U16 KAQY214STLD, U17 KAQY214STLD, U18 KAQY214STLD, U19 KAQY214STLD, U2 KAQY214STLD, U20 KAQY214STLD, U21 KAQY214STLD, U22 KAQY214STLD, U23 KAQY214STLD, U24 KAQY214STLD, U25 KAQY214STLD, U26 KAQY214STLD, U27 KAQY214STLD, U28 KAQY214STLD, U29 KAQY214STLD, U3 KAQY214STLD, U30 KAQY214STLD, U31 KAQY214STLD, U32 KAQY214STLD, U4 KAQY214STLD, U5 KAQY214STLD, U6 KAQY214STLD, U7 KAQY214STLD, U8 KAQY214STLD, U9 KAQY214STLD

Commit message: update
Parts:
- removed the R10 at (8.00, 18.2)
- removed the R11 at (19.2, 16.6)
- removed the R12 at (14.8, 16.6)
- removed the R13 at (10.6, 16.6)
- removed the R14 at (21.8, -16.5)
- removed the R15 at (13.8, -15.8)
- removed the R16 at (17.2, -16.5)
- removed the R17 at (11.0, -18.2)
- added R1: 95.3 1%, Resistor_SMD:R_0603_1608Metric_Pad0.98x0.95mm_HandSolder, F.Cu at (8.10, 18.2)
- added R2: 84.5 1%, Resistor_SMD:R_0603_1608Metric_Pad0.98x0.95mm_HandSolder, F.Cu at (19.2, 16.6)
- added R3: 84.5 1%, Resistor_SMD:R_0603_1608Metric_Pad0.98x0.95mm_HandSolder, F.Cu at (14.8, 16.6)
- added R4: 84.5 1%, Resistor_SMD:R_0603_1608Metric_Pad0.98x0.95mm_HandSolder, F.Cu at (10.6, 16.5)
- added R5: 84.5 1%, Resistor_SMD:R_0603_1608Metric_Pad0.98x0.95mm_HandSolder, F.Cu at (21.8, -16.6)
- added R6: 84.5 1%, Resistor_SMD:R_0603_1608Metric_Pad0.98x0.95mm_HandSolder, F.Cu at (13.8, -15.8)
- added R7: 84.5 1%, Resistor_SMD:R_0603_1608Metric_Pad0.98x0.95mm_HandSolder, F.Cu at (17.2, -16.5)
- added R8: 95.3 1%, Resistor_SMD:R_0603_1608Metric_Pad0.98x0.95mm_HandSolder, F.Cu at (11.1, -18.2)
- C1: value 1uF -> 100nF
- renumbered J5 to J4, J6 to J5, R2 to R10, R3 to R11, R18 to R12, R19 to R13, R20 to R14, R21 to R15, R22 to R16, R23 to R17, R24 to R18, R25 to R19, R26 to R20, R27 to R21, R28 to R22, R29 to R23, R4 to R24, R5 to R25, R6 to R26, R7 to R27, R8 to R28, R9 to R29, R1 to R9, U9 to U10, U10 to U11, U11 to U12, U12 to U13, U13 to U14, U14 to U15, U15 to U16, U16 to U17, U17 to U18, U18 to U19, U19 to U20, U20 to U21, U21 to U22, U22 to U23, U23 to U24, U24 to U25, U25 to U26, U26 to U27, U27 to U28, U28 to U29, U29 to U30, U30 to U31, U31 to U32, U32 to U33, M1 to U9
Connections:
- J2 pad 3: GND -> GNDS
Routing:
- net GNDS: track 30.0 -> 36.2 mm
