File: Calibrator_02/Calibrator_02/Resistor_Network.sch (KiCad schematic (older format))
At the start: 60 parts, among them U10 KAQY214STLD, U11 KAQY214STLD, U12 KAQY214STLD, U13 KAQY214STLD, U14 KAQY214STLD, U15 KAQY214STLD, U16 KAQY214STLD, U17 KAQY214STLD, U18 KAQY214STLD, U19 KAQY214STLD, U20 KAQY214STLD, U21 KAQY214STLD, U22 KAQY214STLD, U23 KAQY214STLD, U24 KAQY214STLD, U25 KAQY214STLD, U26 KAQY214STLD, U27 KAQY214STLD, U28 KAQY214STLD, U29 KAQY214STLD, U30 KAQY214STLD, U31 KAQY214STLD, U32 KAQY214STLD, U9 KAQY214STLD

Commit message: Fixed footprint
Parts:
- R18, R19, R20, R21, R22, R23, R24, R25, R26, R27, R28, R29, R30, R31, R32, R33, R34, R35, R36, R37, R38, R39, R40, R41: footprint Resistor_SMD:R_0201_0603Metric_Pad0.64x0.40mm_HandSolder -> Resistor_SMD:R_0603_1608Metric_Pad0.98x0.95mm_HandSolder
Changed lines of the file:
@@
 F 0 "R18" H 1920 1196 50  0000 L CNN
 F 1 "95.3 1%" H 1920 1105 50  0000 L CNN
-F 2 "Resistor_SMD:R_0201_0603Metric_Pad0.64x0.40mm_HandSolder" V 1780 1150 50  0001 C CNN
+F 2 "Resistor_SMD:R_0603_1608Metric_Pad0.98x0.95mm_HandSolder" V 1780 1150 50  0001 C CNN
 F 3 "~" H 1850 1150 50  0001 C CNN
 F 4 "C218188" H 1850 1150 50  0001 C CNN "LCSC"
@@
 F 0 "R23" H 12070 1196 50  0000 L CNN
 F 1 "95.3 1%" H 12070 1105 50  0000 L CNN
-F 2 "Resistor_SMD:R_0201_0603Metric_Pad0.64x0.40mm_HandSolder" V 11930 1150 50  0001 C CNN
+F 2 "Resistor_SMD:R_0603_1608Metric_Pad0.98x0.95mm_HandSolder" V 11930 1150 50  0001 C CNN
 F 3 "~" H 12000 1150 50  0001 C CNN
 F 4 "C218188" H 12000 1150 50  0001 C CNN "LCSC"
@@
 F 0 "R22" H 10020 1196 50  0000 L CNN
 F 1 "95.3 1%" H 10020 1105 50  0000 L CNN
-F 2 "Resistor_SMD:R_0201_0603Metric_Pad0.64x0.40mm_HandSolder" V 9880 1150 50  0001 C CNN
+F 2 "Resistor_SMD:R_0603_1608Metric_Pad0.98x0.95mm_HandSolder" V 9880 1150 50  0001 C CNN
 F 3 "~" H 9950 1150 50  0001 C CNN
 F 4 "C218188" H 9950 1150 50  0001 C CNN "LCSC"
@@
 F 0 "R21" H 7970 1196 50  0000 L CNN
 F 1 "95.3 1%" H 7970 1105 50  0000 L CNN
-F 2 "Resistor_SMD:R_0201_0603Metric_Pad0.64x0.40mm_HandSolder" V 7830 1150 50  0001 C CNN
+F 2 "Resistor_SMD:R_0603_1608Metric_Pad0.98x0.95mm_HandSolder" V 7830 1150 50  0001 C CNN
 F 3 "~" H 7900 1150 50  0001 C CNN
 F 4 "C218188" H 7900 1150 50  0001 C CNN "LCSC"
@@
 F 0 "R20" H 5970 1196 50  0000 L CNN
 F 1 "95.3 1%" H 5970 1105 50  0000 L CNN
-F 2 "Resistor_SMD:R_0201_0603Metric_Pad0.64x0.40mm_HandSolder" V 5830 1150 50  0001 C CNN
+F 2 "Resistor_SMD:R_0603_1608Metric_Pad0.98x0.95mm_HandSolder" V 5830 1150 50  0001 C CNN
 F 3 "~" H 5900 1150 50  0001 C CNN
 F 4 "C218188" H 5900 1150 50  0001 C CNN "LCSC"
@@
 F 0 "R19" H 3970 1196 50  0000 L CNN
 F 1 "95.3 1%" H 3970 1105 50  0000 L CNN
-F 2 "Resistor_SMD:R_0201_0603Metric_Pad0.64x0.40mm_HandSolder" V 3830 1150 50  0001 C CNN
+F 2 "Resistor_SMD:R_0603_1608Metric_Pad0.98x0.95mm_HandSolder" V 3830 1150 50  0001 C CNN
 F 3 "~" H 3900 1150 50  0001 C CNN
 F 4 "C218188" H 3900 1150 50  0001 C CNN "LCSC"
@@
 F 0 "R24" H 2820 1496 50  0000 L CNN
 F 1 "84.5 1%" H 2820 1405 50  0000 L CNN
-F 2 "Resistor_SMD:R_0201_0603Metric_Pad0.64x0.40mm_HandSolder" V 2680 1450 50  0001 C CNN
+F 2 "Resistor_SMD:R_0603_1608Metric_Pad0.98x0.95mm_HandSolder" V 2680 1450 50  0001 C CNN
 F 3 "~" H 2750 1450 50  0001 C CNN
 F 4 "C177824" H 2750 1450 50  0001 C CNN "LCSC"
@@
 F 0 "R25" H 4870 1496 50  0000 L CNN
 F 1 "84.5 1%" H 4870 1405 50  0000 L CNN
-F 2 "Resistor_SMD:R_0201_0603Metric_Pad0.64x0.40mm_HandSolder" V 4730 1450 50  0001 C CNN
+F 2 "Resistor_SMD:R_0603_1608Metric_Pad0.98x0.95mm_HandSolder" V 4730 1450 50  0001 C CNN
 F 3 "~" H 4800 1450 50  0001 C CNN
 F 4 "C177824" H 4800 1450 50  0001 C CNN "LCSC"
@@
 F 0 "R26" H 6870 1496 50  0000 L CNN
 F 1 "84.5 1%" H 6870 1405 50  0000 L CNN
-F 2 "Resistor_SMD:R_0201_0603Metric_Pad0.64x0.40mm_HandSolder" V 6730 1450 50  0001 C CNN
+F 2 "Resistor_SMD:R_0603_1608Metric_Pad0.98x0.95mm_HandSolder" V 6730 1450 50  0001 C CNN
 F 3 "~" H 6800 1450 50  0001 C CNN
 F 4 "C177824" H 6800 1450 50  0001 C CNN "LCSC"
@@
 F 0 "R27" H 8870 1496 50  0000 L CNN
 F 1 "84.5 1%" H 8870 1405 50  0000 L CNN
-F 2 "Resistor_SMD:R_0201_0603Metric_Pad0.64x0.40mm_HandSolder" V 8730 1450 50  0001 C CNN
+F 2 "Resistor_SMD:R_0603_1608Metric_Pad0.98x0.95mm_HandSolder" V 8730 1450 50  0001 C CNN
 F 3 "~" H 8800 1450 50  0001 C CNN
 F 4 "C177824" H 8800 1450 50  0001 C CNN "LCSC"
@@
 F 0 "R28" H 10920 1496 50  0000 L CNN
 F 1 "84.5 1%" H 10920 1405 50  0000 L CNN
-F 2 "Resistor_SMD:R_0201_0603Metric_Pad0.64x0.40mm_HandSolder" V 10780 1450 50  0001 C CNN
+F 2 "Resistor_SMD:R_0603_1608Metric_Pad0.98x0.95mm_HandSolder" V 10780 1450 50  0001 C CNN
 F 3 "~" H 10850 1450 50  0001 C CNN
 F 4 "C177824" H 10850 1450 50  0001 C CNN "LCSC"
@@
 F 0 "R29" H 12970 1496 50  0000 L CNN
 F 1 "84.5 1%" H 12970 1405 50  0000 L CNN
-F 2 "Resistor_SMD:R_0201_0603Metric_Pad0.64x0.40mm_HandSolder" V 12830 1450 50  0001 C CNN
+F 2 "Resistor_SMD:R_0603_1608Metric_Pad0.98x0.95mm_HandSolder" V 12830 1450 50  0001 C CNN
 F 3 "~" H 12900 1450 50  0001 C CNN
 F 4 "C177824" H 12900 1450 50  0001 C CNN "LCSC"
@@
 F 0 "R41" H 12420 4996 50  0000 L CNN
 F 1 "84.5 1%" H 12420 4905 50  0000 L CNN
-F 2 "Resistor_SMD:R_0201_0603Metric_Pad0.64x0.40mm_HandSolder" V 12280 4950 50  0001 C CNN
+F 2 "Resistor_SMD:R_0603_1608Metric_Pad0.98x0.95mm_HandSolder" V 12280 4950 50  0001 C CNN
 F 3 "~" H 12350 4950 50  0001 C CNN
 F 4 "C177824" H 12350 4950 50  0001 C CNN "LCSC"
@@
 F 0 "R40" H 11520 4996 50  0000 L CNN
 F 1 "84.5 1%" H 11520 4905 50  0000 L CNN
-F 2 "Resistor_SMD:R_0201_0603Metric_Pad0.64x0.40mm_HandSolder" V 11380 4950 50  0001 C CNN
+F 2 "Resistor_SMD:R_0603_1608Metric_Pad0.98x0.95mm_HandSolder" V 11380 4950 50  0001 C CNN
 F 3 "~" H 11450 4950 50  0001 C CNN
 F 4 "C177824" H 11450 4950 50  0001 C CNN "LCSC"
@@
 F 0 "R39" H 10370 4996 50  0000 L CNN
 F 1 "84.5 1%" H 10370 4905 50  0000 L CNN
-F 2 "Resistor_SMD:R_0201_0603Metric_Pad0.64x0.40mm_HandSolder" V 10230 4950 50  0001 C CNN
+F 2 "Resistor_SMD:R_0603_1608Metric_Pad0.98x0.95mm_HandSolder" V 10230 4950 50  0001 C CNN
 F 3 "~" H 10300 4950 50  0001 C CNN
 F 4 "C177824" H 10300 4950 50  0001 C CNN "LCSC"
@@
 F 0 "R38" H 9470 4996 50  0000 L CNN
 F 1 "84.5 1%" H 9470 4905 50  0000 L CNN
-F 2 "Resistor_SMD:R_0201_0603Metric_Pad0.64x0.40mm_HandSolder" V 9330 4950 50  0001 C CNN
+F 2 "Resistor_SMD:R_0603_1608Metric_Pad0.98x0.95mm_HandSolder" V 9330 4950 50  0001 C CNN
 F 3 "~" H 9400 4950 50  0001 C CNN
 F 4 "C177824" H 9400 4950 50  0001 C CNN "LCSC"
@@
 F 0 "R37" H 8270 4996 50  0000 L CNN
 F 1 "84.5 1%" H 8270 4905 50  0000 L CNN
-F 2 "Resistor_SMD:R_0201_0603Metric_Pad0.64x0.40mm_HandSolder" V 8130 4950 50  0001 C CNN
+F 2 "Resistor_SMD:R_0603_1608Metric_Pad0.98x0.95mm_HandSolder" V 8130 4950 50  0001 C CNN
 F 3 "~" H 8200 4950 50  0001 C CNN
 F 4 "C177824" H 8200 4950 50  0001 C CNN "LCSC"
@@
 F 0 "R36" H 7370 4996 50  0000 L CNN
 F 1 "84.5 1%" H 7370 4905 50  0000 L CNN
-F 2 "Resistor_SMD:R_0201_0603Metric_Pad0.64x0.40mm_HandSolder" V 7230 4950 50  0001 C CNN
+F 2 "Resistor_SMD:R_0603_1608Metric_Pad0.98x0.95mm_HandSolder" V 7230 4950 50  0001 C CNN
 F 3 "~" H 7300 4950 50  0001 C CNN
 F 4 "C177824" H 7300 4950 50  0001 C CNN "LCSC"
@@
 F 0 "R35" H 6320 4996 50  0000 L CNN
 F 1 "84.5 1%" H 6320 4905 50  0000 L CNN
-F 2 "Resistor_SMD:R_0201_0603Metric_Pad0.64x0.40mm_HandSolder" V 6180 4950 50  0001 C CNN
+F 2 "Resistor_SMD:R_0603_1608Metric_Pad0.98x0.95mm_HandSolder" V 6180 4950 50  0001 C CNN
 F 3 "~" H 6250 4950 50  0001 C CNN
 F 4 "C177824" H 6250 4950 50  0001 C CNN "LCSC"
@@
 F 0 "R34" H 5420 4996 50  0000 L CNN
 F 1 "84.5 1%" H 5420 4905 50  0000 L CNN
-F 2 "Resistor_SMD:R_0201_0603Metric_Pad0.64x0.40mm_HandSolder" V 5280 4950 50  0001 C CNN
+F 2 "Resistor_SMD:R_0603_1608Metric_Pad0.98x0.95mm_HandSolder" V 5280 4950 50  0001 C CNN
 F 3 "~" H 5350 4950 50  0001 C CNN
 F 4 "C177824" H 5350 4950 50  0001 C CNN "LCSC"
@@
 F 0 "R33" H 4320 4996 50  0000 L CNN
 F 1 "84.5 1%" H 4320 4905 50  0000 L CNN
-F 2 "Resistor_SMD:R_0201_0603Metric_Pad0.64x0.40mm_HandSolder" V 4180 4950 50  0001 C CNN
+F 2 "Resistor_SMD:R_0603_1608Metric_Pad0.98x0.95mm_HandSolder" V 4180 4950 50  0001 C CNN
 F 3 "~" H 4250 4950 50  0001 C CNN
 F 4 "C177824" H 4250 4950 50  0001 C CNN "LCSC"
@@
 F 0 "R32" H 3420 4996 50  0000 L CNN
 F 1 "84.5 1%" H 3420 4905 50  0000 L CNN
-F 2 "Resistor_SMD:R_0201_0603Metric_Pad0.64x0.40mm_HandSolder" V 3280 4950 50  0001 C CNN
+F 2 "Resistor_SMD:R_0603_1608Metric_Pad0.98x0.95mm_HandSolder" V 3280 4950 50  0001 C CNN
 F 3 "~" H 3350 4950 50  0001 C CNN
 F 4 "C177824" H 3350 4950 50  0001 C CNN "LCSC"
@@
 F 0 "R31" H 2220 4996 50  0000 L CNN
 F 1 "84.5 1%" H 2220 4905 50  0000 L CNN
-F 2 "Resistor_SMD:R_0201_0603Metric_Pad0.64x0.40mm_HandSolder" V 2080 4950 50  0001 C CNN
+F 2 "Resistor_SMD:R_0603_1608Metric_Pad0.98x0.95mm_HandSolder" V 2080 4950 50  0001 C CNN
 F 3 "~" H 2150 4950 50  0001 C CNN
 F 4 "C177824" H 2150 4950 50  0001 C CNN "LCSC"
@@
 F 0 "R30" H 1320 4996 50  0000 L CNN
 F 1 "84.5 1%" H 1320 4905 50  0000 L CNN
-F 2 "Resistor_SMD:R_0201_0603Metric_Pad0.64x0.40mm_HandSolder" V 1180 4950 50  0001 C CNN
+F 2 "Resistor_SMD:R_0603_1608Metric_Pad0.98x0.95mm_HandSolder" V 1180 4950 50  0001 C CNN
 F 3 "~" H 1250 4950 50  0001 C CNN
 F 4 "C177824" H 1250 4950 50  0001 C CNN "LCSC"

Commit message: update
Parts:
- renumbered R18 to R12, R19 to R13, R20 to R14, R21 to R15, R22 to R16, R23 to R17, R24 to R18, R25 to R19, R26 to R20, R27 to R21, R28 to R22, R29 to R23, R4 to R24, R5 to R25, R6 to R26, R7 to R27, R8 to R28, R9 to R29, U9 to U10, U10 to U11, U11 to U12, U12 to U13, U13 to U14, U14 to U15, U15 to U16, U16 to U17, U17 to U18, U18 to U19, U19 to U20, U20 to U21, U21 to U22, U22 to U23, U23 to U24, U24 to U25, U25 to U26, U26 to U27, U27 to U28, U28 to U29, U29 to U30, U30 to U31, U31 to U32, U32 to U33
